File: pi-ups/high-side-simple/pi-ups-high-simple.sch (KiCad schematic (older format))
At the start: 15 parts, among them J1 USB_A, J2 USB_A, J3 USB_A, Q3 IRLM2244, Q4 IRLM2244, U1 DC-DC Converter

Commit message: Beautify
Connections:
- wire segments 64 -> 62
Changed lines of the file:
@@
 EESchema Schematic File Version 4
+LIBS:pi-ups-high-simple-cache
 EELAYER 26 0
 EELAYER END
@@
 $EndComp
 Wire Wire Line
-	2900 2400 2900 2350
-Wire Wire Line
-	2900 2050 2900 2000
-Wire Wire Line
 	5150 1550 5150 1950
