File: nixie-clock-v2/nixie-clock-v2/nixie-clock-v2.sch (KiCad schematic (older format))
At the start: 7 parts

Commit message: wip
Parts:
- removed N? (x6): IN-8-2, russian-nixies-IN-8-2, symbol russian-nixies:IN-8-2
- removed U?: Arduino_Pro_Mini, symbol microfarad-de:Arduino_Pro_Mini
- added N? (x2): IN-8-2, russian-nixies-IN-8-2, symbol russian-nixies:IN-8-2
- added R? (x2): R, symbol Device:R
- added U? (x2): TLP127, Package_SO:MFSOP6-4_4.4x3.6mm_P1.27mm, symbol Isolator:TLP127
- added U? (x3): TPIC6595, symbol Interface_Expansion:TPIC6595
- added U?: Arduino_Pro_Mini, symbol microfarad-de:Arduino_Pro_Mini
Connections:
- new net: N?.A, U?.4 (x2)
- new net: R?.2, U?.6 (x2)
- new net: N?.. (RHDP), U?.15 (DRAIN5)
- new net: N?.0, U?.14 (DRAIN4)
- new net: N?.1, U?.7 (DRAIN3)
- new net: N?.2, U?.14 (DRAIN4)
- new net: N?.3, U?.15 (DRAIN5)
- new net: N?.4, U?.16 (DRAIN6)
- new net: N?.5, U?.17 (DRAIN7)
- new net: N?.6, U?.4 (DRAIN0)
- new net: N?.7, U?.5 (DRAIN1)
- new net: N?.8, U?.6 (DRAIN2)
- new net: N?.9, U?.7 (DRAIN3)
- new net: N?.. (RHDP), U?.6 (DRAIN2)
- new net: N?.0, U?.5 (DRAIN1)
- new net: N?.1, U?.4 (DRAIN0)
- new net: N?.2, U?.5 (DRAIN1)
- new net: N?.3, U?.6 (DRAIN2)
- new net: N?.4, U?.7 (DRAIN3)
- new net: N?.5, U?.14 (DRAIN4)
- new net: N?.6, U?.15 (DRAIN5)
- new net: N?.7, U?.16 (DRAIN6)
- new net: N?.8, U?.17 (DRAIN7)
- new net: N?.9, U?.4 (DRAIN0)
- new net: U?.18 (SER_OUT), U?.3 (SER_IN) (x2)
- new net +5V: U?.2 (VCC), U?.2 (VCC), U?.2 (VCC)
- new net GND: U?.1 (PGND), U?.1 (PGND), U?.1 (PGND), U?.10 (PGND), U?.10 (PGND), U?.10 (PGND), U?.11 (PGND), U?.11 (PGND), U?.11 (PGND), U?.19 (LGND), U?.19 (LGND), U?.19 (LGND), U?.20 (PGND), U?.20 (PGND), U?.20 (PGND), U?.3, U?.3
