File: brush-timer/brush-timer.sch (KiCad schematic (older format))
At the start: 13 parts, among them Q1 BC327, Q2 BC337, SW1 Power, U1 Arduino_Pro_Mini

Commit message: Updated brush-timer.sch
Parts:
- removed C1: 100µF, symbol Device:CP
- added R?: 1M, symbol Device:R
- R1: value 220K -> 1M
- R2, R3: value 56K -> 100K
Connections:
- net GND: now also R?.2
- net at Q2.2 (B), R3.2: now also R?.1
Other:
- moved on the sheet: R2, R3
Changed lines of the file:
@@
 P 2250 2400
 F 0 "R1" H 2320 2446 50  0000 L CNN
-F 1 "220K" H 2320 2355 50  0000 L CNN
+F 1 "1M" H 2320 2355 50  0000 L CNN
 F 2 "" V 2180 2400 50  0001 C CNN
 F 3 "~" H 2250 2400 50  0001 C CNN
@@
 L Device:R R2
 U 1 1 5C6AFDBA
-P 2650 2150
-F 0 "R2" V 2443 2150 50  0000 C CNN
-F 1 "56K" V 2534 2150 50  0000 C CNN
-F 2 "" V 2580 2150 50  0001 C CNN
-F 3 "~" H 2650 2150 50  0001 C CNN
-	1    2650 2150
+P 2600 2150
+F 0 "R2" V 2393 2150 50  0000 C CNN
+F 1 "100K" V 2484 2150 50  0000 C CNN
+F 2 "" V 2530 2150 50  0001 C CNN
+F 3 "~" H 2600 2150 50  0001 C CNN
+	1    2600 2150
 	0    1    1    0
 $EndComp
 Wire Wire Line
-	2250 2150 2500 2150
+	2250 2150 2450 2150
 Wire Wire Line
 	2900 2150 2900 2250
 Wire Wire Line
-	2800 2150 2900 2150
+	2750 2150 2900 2150
 Wire Wire Line
 	2250 2250 2250 2150
@@
 L Device:R R3
 U 1 1 5C6B03EE
-P 4150 2450
-F 0 "R3" V 4250 2450 50  0000 C CNN
-F 1 "56K" V 4350 2450 50  0000 C CNN
-F 2 "" V 4080 2450 50  0001 C CNN
-F 3 "~" H 4150 2450 50  0001 C CNN
-	1    4150 2450
+P 3550 2450
+F 0 "R3" V 3650 2450 50  0000 C CNN
+F 1 "100K" V 3750 2450 50  0000 C CNN
+F 2 "" V 3480 2450 50  0001 C CNN
+F 3 "~" H 3550 2450 50  0001 C CNN
+	1    3550 2450
 	0    1    1    0
 $EndComp
 Wire Wire Line
-	3200 2450 4000 2450
+	3200 2450 3400 2450
 $Comp
 L power:GND #PWR03
@@
 $EndComp
 Wire Wire Line
-	2900 3300 2900 2650
+	2900 3300 2900 2900
 $Comp
 L Switch:SW_Push SW1
@@
 $EndComp
 Wire Wire Line
-	4300 2450 5100 2450
+	3700 2450 5100 2450
 Wire Wire Line
 	2250 2150 2250 1550
@@
 L power:VCC #PWR06
 U 1 1 5C6B316B
-P 4700 1350
-F 0 "#PWR06" H 4700 1200 50  0001 C CNN
-F 1 "VCC" H 4717 1523 50  0000 C CNN
-F 2 "" H 4700 1350 50  0001 C CNN
-F 3 "" H 4700 1350 50  0001 C CNN
-	1    4700 1350
-	1    0    0    -1
-$EndComp
-Wire Wire Line
-	4700 1350 4700 1750
-Wire Wire Line
-	4700 1750 5100 1750
+P 4850 1350
+F 0 "#PWR06" H 4850 1200 50  0001 C CNN
+F 1 "VCC" H 4867 1523 50  0000 C CNN
+F 2 "" H 4850 1350 50  0001 C CNN
+F 3 "" H 4850 1350 50  0001 C CNN
+	1    4850 1350
+	1    0    0    -1
+$EndComp
+Wire Wire Line
+	4850 1350 4850 1750
+Wire Wire Line
+	4850 1750 5100 1750
 $Comp
 L power:GND #PWR08
@@
 	4600 3300 4600 3250
 $Comp
-L Device:CP C1
-U 1 1 5C6B4ED8
-P 4700 1900
-F 0 "C1" H 4818 1946 50  0000 L CNN
-F 1 "100µF" H 4818 1855 50  0000 L CNN
-F 2 "" H 4738 1750 50  0001 C CNN
-F 3 "~" H 4700 1900 50  0001 C CNN
-	1    4700 1900
-	1    0    0    -1
-$EndComp
-Connection ~ 4700 1750
-$Comp
-L power:GND #PWR07
-U 1 1 5C6B5B7A
-P 4700 2050
-F 0 "#PWR07" H 4700 1800 50  0001 C CNN
-F 1 "GND" H 4700 1900 50  0000 C CNN
-F 2 "" H 4700 2050 50  0001 C CNN
-F 3 "" H 4700 2050 50  0001 C CNN
-	1    4700 2050
-	1    0    0    -1
-$EndComp
+L Device:R R?
+U 1 1 5C6B7A97
+P 3200 2700
+F 0 "R?" H 3270 2746 50  0000 L CNN
+F 1 "1M" H 3270 2655 50  0000 L CNN
+F 2 "" V 3130 2700 50  0001 C CNN
+F 3 "~" H 3200 2700 50  0001 C CNN
+	1    3200 2700
+	1    0    0    -1
+$EndComp
+Wire Wire Line
+	3200 2550 3200 2450
+Connection ~ 3200 2450
+Wire Wire Line
+	3200 2850 3200 2900
+Wire Wire Line
+	3200 2900 2900 2900
+Connection ~ 2900 2900
+Wire Wire Line
+	2900 2900 2900 2650
 $EndSCHEMATC

Commit message: Update brush-timer.sch
Parts:
- gave numbers to parts that had none: 1
- renumbered R3 to R4, R4 to R5
Changed lines of the file:
@@
 	1950 1350 1950 1950
 $Comp
-L Device:R R3
+L Device:R R4
 U 1 1 5C6B03EE
 P 3550 2450
-F 0 "R3" V 3650 2450 50  0000 C CNN
+F 0 "R4" V 3650 2450 50  0000 C CNN
 F 1 "100K" V 3750 2450 50  0000 C CNN
 F 2 "" V 3480 2450 50  0001 C CNN
@@
 	4850 1750 5100 1750
 $Comp
-L power:GND #PWR08
+L power:GND #PWR07
 U 1 1 5C6B344C
 P 6350 2050
-F 0 "#PWR08" H 6350 1800 50  0001 C CNN
+F 0 "#PWR07" H 6350 1800 50  0001 C CNN
 F 1 "GND" H 6355 1877 50  0000 C CNN
 F 2 "" H 6350 2050 50  0001 C CNN
@@
 $EndComp
 $Comp
-L Device:R R4
+L Device:R R5
 U 1 1 5C6B37B0
 P 4600 2750
-F 0 "R4" H 4670 2796 50  0000 L CNN
+F 0 "R5" H 4670 2796 50  0000 L CNN
 F 1 "1K5" H 4670 2705 50  0000 L CNN
 F 2 "" V 4530 2750 50  0001 C CNN
@@
 	4600 3300 4600 3250
 $Comp
-L Device:R R?
+L Device:R R3
 U 1 1 5C6B7A97
 P 3200 2700
-F 0 "R?" H 3270 2746 50  0000 L CNN
+F 0 "R3" H 3270 2746 50  0000 L CNN
 F 1 "1M" H 3270 2655 50  0000 L CNN
 F 2 "" V 3130 2700 50  0001 C CNN
