File: brush-timer/brush-timer.sch (KiCad schematic (older format))
At the start: 20 parts, among them Q1 IRL2244, Q2 IRL6244, SW1 Power, U1 Arduino_Pro_Mini

Commit message: Update brush-timer.sch
Parts:
- R5: value 820R -> 2K2
Changed lines of the file:
@@
 P 6350 3600
 F 0 "R5" H 6420 3646 50  0000 L CNN
-F 1 "820R" H 6420 3555 50  0000 L CNN
+F 1 "2K2" H 6420 3555 50  0000 L CNN
 F 2 "" V 6280 3600 50  0001 C CNN
 F 3 "~" H 6350 3600 50  0001 C CNN

Commit message: Updated brush-timer.sh
Parts:
- removed JP1: Program, symbol Device:Jumper
Changed lines of the file:
@@
 Sheet 1 1
 Title "Arduino Toothbrush Timer"
-Date "2019-02-20"
+Date "2019-02-21"
 Rev ""
 Comp "microfarad.de"
@@
 Connection ~ 1350 1900
 Wire Wire Line
-	1350 1900 1550 1900
-Wire Wire Line
 	2700 1700 2700 1800
 Wire Wire Line
@@
 Wire Wire Line
 	7150 1600 7150 2950
-$Comp
-L Device:Jumper JP1
-U 1 1 5C6D3EE3
-P 1550 2650
-F 0 "JP1" V 1504 2776 50  0000 L CNN
-F 1 "Program" V 1595 2776 50  0000 L CNN
-F 2 "" H 1550 2650 50  0001 C CNN
-F 3 "~" H 1550 2650 50  0001 C CNN
-	1    1550 2650
-	0    1    1    0
-$EndComp
-Wire Wire Line
-	1550 2350 1550 1900
-Connection ~ 1550 1900
-Wire Wire Line
-	1550 1900 2000 1900
-$Comp
-L power:GND #PWR08
-U 1 1 5C6D7A03
-P 1550 3050
-F 0 "#PWR08" H 1550 2800 50  0001 C CNN
-F 1 "GND" H 1555 2877 50  0000 C CNN
-F 2 "" H 1550 3050 50  0001 C CNN
-F 3 "" H 1550 3050 50  0001 C CNN
-	1    1550 3050
-	1    0    0    -1
-$EndComp
-Wire Wire Line
-	1550 3050 1550 2950
 Wire Wire Line
 	4200 1300 4100 1300
@@
 Wire Wire Line
 	3950 1100 3950 1200
+Wire Wire Line
+	1350 1900 2000 1900
 $EndSCHEMATC
