File: toothbrush-timer/toothbrush-timer.sch (KiCad schematic (older format))
At the start: 19 parts, among them Q1 IRL2244, Q2 IRL6244, SW1 Power, U1 Arduino_Pro_Mini

Commit message: Updated toohtbrush-timer
Parts:
- Q1: value IRL2244 -> IRLML2244
- Q2: value IRL6244 -> IRLML6244
Changed lines of the file:
@@
 F 3 "~" H 1350 2150 50  0001 C CNN
 	1    1350 2150
-	1    0    0    -1
+	-1   0    0    -1
 $EndComp
 $Comp
@@
 P 2100 2200
 F 0 "Q2" H 2306 2246 50  0000 L CNN
-F 1 "IRL6244" H 2306 2155 50  0000 L CNN
+F 1 "IRLML6244" H 2306 2155 50  0000 L CNN
 F 2 "" H 2300 2300 50  0001 C CNN
 F 3 "~" H 2100 2200 50  0001 C CNN
@@
 P 1150 1900
 F 0 "Q1" H 1356 1946 50  0000 L CNN
-F 1 "IRL2244" H 1356 1855 50  0000 L CNN
+F 1 "IRLML2244" H 1356 1855 50  0000 L CNN
 F 2 "" H 1350 2000 50  0001 C CNN
 F 3 "~" H 1150 1900 50  0001 C CNN

Commit message: Updated toothbrush-timer
Parts:
- renumbered R3 to R2, R5 to R3
Changed lines of the file:
@@
 EESchema Schematic File Version 4
+LIBS:toothbrush-timer-cache
 EELAYER 26 0
 EELAYER END
@@
 Sheet 1 1
 Title "Arduino Toothbrush Timer"
-Date "2019-02-21"
+Date "2019-03-22"
 Rev ""
 Comp "microfarad.de"
@@
 $EndComp
 $Comp
-L power:VCC #PWR06
+L power:VCC #PWR05
 U 1 1 5C6B316B
 P 3750 1100
-F 0 "#PWR06" H 3750 950 50  0001 C CNN
+F 0 "#PWR05" H 3750 950 50  0001 C CNN
 F 1 "VCC" H 3767 1273 50  0000 C CNN
 F 2 "" H 3750 1100 50  0001 C CNN
@@
 	3750 1500 4200 1500
 $Comp
-L power:GND #PWR07
+L power:GND #PWR06
 U 1 1 5C6B344C
 P 3950 1200
-F 0 "#PWR07" H 3950 950 50  0001 C CNN
+F 0 "#PWR06" H 3950 950 50  0001 C CNN
 F 1 "GND" H 3955 1027 50  0000 C CNN
 F 2 "" H 3950 1200 50  0001 C CNN
@@
 $EndComp
 $Comp
-L Device:R R5
+L Device:R R3
 U 1 1 5C6B37B0
 P 6350 3600
-F 0 "R5" H 6420 3646 50  0000 L CNN
+F 0 "R3" H 6420 3646 50  0000 L CNN
 F 1 "2K2" H 6420 3555 50  0000 L CNN
 F 2 "" V 6280 3600 50  0001 C CNN
@@
 $EndComp
 $Comp
-L power:GND #PWR05
+L power:GND #PWR07
 U 1 1 5C6B44BA
 P 6350 3800
-F 0 "#PWR05" H 6350 3550 50  0001 C CNN
+F 0 "#PWR07" H 6350 3550 50  0001 C CNN
 F 1 "GND" H 6355 3627 50  0000 C CNN
 F 2 "" H 6350 3800 50  0001 C CNN
@@
 $EndComp
 $Comp
-L Device:R R3
+L Device:R R2
 U 1 1 5C6B7A97
 P 2300 2450
-F 0 "R3" H 2370 2496 50  0000 L CNN
+F 0 "R2" H 2370 2496 50  0000 L CNN
 F 1 "1M" H 2370 2405 50  0000 L CNN
 F 2 "" V 2230 2450 50  0001 C CNN
