File: pi-ups/pi-ups.sch (KiCad schematic (older format))
At the start: 30 parts, among them J1 , Q1 IRLML2244, Q2 IRLML2244, Q3 IRLML2244, Q4 IRLML2244, U1 BMS_1S, U2 DC-DC, U3 BMS_1S, U4 FTDI232, U5 Arduino_Pro_Mini

Commit message: pi-ups: separate RPi and HDD outputs, filter capacitors
Parts:
- added C1, C2: 220nF, symbol Device:C
- added C3: 47µF/50V, symbol Device:CP
- added C5: 470nF, symbol Device:C
- renumbered C1 to C4, C2 to C6, C3 to C7
Connections:
- net +5V: now also C1.1
- net GND: now also C1.2, C2.2, C3.2, C5.1
- net V_IN: now also C5.2
- net V_RPI: now also C2.1, C3.1
Other:
- moved on the sheet: U2
Changed lines of the file:
@@
 $EndComp
 $Comp
-L power:GND #PWR09
+L power:GND #PWR06
 U 1 1 5CDDD224
 P 5700 4850
-F 0 "#PWR09" H 5700 4600 50  0001 C CNN
+F 0 "#PWR06" H 5700 4600 50  0001 C CNN
 F 1 "GND" H 5705 4677 50  0000 C CNN
 F 2 "" H 5700 4850 50  0001 C CNN
@@
 $EndComp
 $Comp
-L Device:C C1
+L Device:C C4
 U 1 1 5CDDD4BF
 P 5700 5350
-F 0 "C1" V 5950 5400 50  0000 R CNN
+F 0 "C4" V 5950 5400 50  0000 R CNN
 F 1 "100n" V 5850 5400 50  0000 R CNN
 F 2 "" H 5738 5200 50  0001 C CNN
@@
 	2300 1550 2200 1550
 $Comp
-L power:GND #PWR03
+L power:GND #PWR02
 U 1 1 5CDDF417
-P 2300 1850
-F 0 "#PWR03" H 2300 1600 50  0001 C CNN
-F 1 "GND" H 2305 1677 50  0000 C CNN
-F 2 "" H 2300 1850 50  0001 C CNN
-F 3 "" H 2300 1850 50  0001 C CNN
-	1    2300 1850
-	1    0    0    -1
-$EndComp
-Text GLabel 2550 1750 2    50   Output ~ 0
+P 2300 2250
+F 0 "#PWR02" H 2300 2000 50  0001 C CNN
+F 1 "GND" H 2305 2077 50  0000 C CNN
+F 2 "" H 2300 2250 50  0001 C CNN
+F 3 "" H 2300 2250 50  0001 C CNN
+	1    2300 2250
+	1    0    0    -1
+$EndComp
+Text GLabel 3450 1750 2    50   Output ~ 0
 V_IN
 Wire Wire Line
-	2300 1850 2300 1650
+	2300 2250 2300 2200
 Connection ~ 2300 1650
 Wire Wire Line
@@
 	2300 1250 2300 1550
 Connection ~ 2300 1550
-Text GLabel 2550 1350 2    50   Input ~ 0
+Text GLabel 3400 1350 2    50   Input ~ 0
 V_RPI
 Wire Wire Line
-	2200 1750 2550 1750
+	2200 1750 3450 1750
 $Comp
 L Device:Battery_Cell BT1
@@
 Connection ~ 2900 4500
 $Comp
-L power:GND #PWR04
+L power:GND #PWR03
 U 1 1 5CDE33F8
 P 2650 5700
-F 0 "#PWR04" H 2650 5450 50  0001 C CNN
+F 0 "#PWR03" H 2650 5450 50  0001 C CNN
 F 1 "GND" H 2655 5527 50  0000 C CNN
 F 2 "" H 2650 5700 50  0001 C CNN
@@
 Wire Wire Line
 	5450 4850 5700 4850
-Text GLabel 3200 2750 2    50   Output ~ 0
+Text GLabel 3200 2850 2    50   Output ~ 0
 V_UPS
 Wire Wire Line
@@
 $EndComp
 $Comp
-L power:+5V #PWR017
+L power:+5V #PWR014
 U 1 1 5CDF6DD4
 P 9700 1350
-F 0 "#PWR017" H 9700 1200 50  0001 C CNN
+F 0 "#PWR014" H 9700 1200 50  0001 C CNN
 F 1 "+5V" H 9715 1523 50  0000 C CNN
 F 2 "" H 9700 1350 50  0001 C CNN
@@
 $EndComp
 $Comp
-L power:+5V #PWR010
+L power:+5V #PWR07
 U 1 1 5CE042BB
 P 6250 2650
-F 0 "#PWR010" H 6250 2500 50  0001 C CNN
+F 0 "#PWR07" H 6250 2500 50  0001 C CNN
 F 1 "+5V" H 6265 2823 50  0000 C CNN
 F 2 "" H 6250 2650 50  0001 C CNN
@@
 $EndComp
 $Comp
-L power:GND #PWR011
+L power:GND #PWR08
 U 1 1 5CE04E5A
 P 7900 2600
-F 0 "#PWR011" H 7900 2350 50  0001 C CNN
+F 0 "#PWR08" H 7900 2350 50  0001 C CNN
 F 1 "GND" H 7900 2450 50  0000 C CNN
 F 2 "" H 7900 2600 50  0001 C CNN
@@
 $EndComp
 $Comp
-L Device:CP C2
+L Device:CP C6
 U 1 1 5CE05AE7
 P 9450 3650
-F 0 "C2" H 9568 3696 50  0000 L CNN
+F 0 "C6" H 9568 3696 50  0000 L CNN
 F 1 "1000µF/10V" H 9568 3605 50  0000 L CNN
 F 2 "" H 9488 3500 50  0001 C CNN
@@
 $EndComp
 $Comp
-L Device:C C3
+L Device:C C7
 U 1 1 5CE05C0B
 P 9950 3650
-F 0 "C3" H 9835 3696 50  0000 R CNN
+F 0 "C7" H 9835 3696 50  0000 R CNN
 F 1 "220nF" H 9835 3605 50  0000 R CNN
 F 2 "" H 9988 3500 50  0001 C CNN
@@
 	9700 3200 9150 3200
 $Comp
-L power:GND #PWR018
+L power:GND #PWR015
 U 1 1 5CE0B0C6
 P 9700 4000
-F 0 "#PWR018" H 9700 3750 50  0001 C CNN
+F 0 "#PWR015" H 9700 3750 50  0001 C CNN
 F 1 "GND" H 9705 3827 50  0000 C CNN
 F 2 "" H 9700 4000 50  0001 C CNN
@@
 L microfarad-de:DC-DC U2
 U 1 1 5CE2F444
-P 2600 2850
-F 0 "U2" H 2600 2850 50  0000 C CNN
-F 1 "DC-DC" H 2600 2750 50  0000 C CNN
-F 2 "" H 3150 3250 50  0001 C CNN
-F 3 "" H 3150 3250 50  0001 C CNN
-	1    2600 2850
-	1    0    0    -1
-$EndComp
-Wire Wire Line
-	3100 2750 3200 2750
-$Comp
-L power:GND #PWR06
+P 2600 2950
+F 0 "U2" H 2600 2950 50  0000 C CNN
+F 1 "DC-DC" H 2600 2850 50  0000 C CNN
+F 2 "" H 3150 3350 50  0001 C CNN
+F 3 "" H 3150 3350 50  0001 C CNN
+	1    2600 2950
+	1    0    0    -1
+$EndComp
+Wire Wire Line
+	3100 2850 3200 2850
+$Comp
+L power:GND #PWR04
 U 1 1 5CE349CD
-P 3200 3050
-F 0 "#PWR06" H 3200 2800 50  0001 C CNN
-F 1 "GND" H 3205 2877 50  0000 C CNN
-F 2 "" H 3200 3050 50  0001 C CNN
-F 3 "" H 3200 3050 50  0001 C CNN
-	1    3200 3050
-	1    0    0    -1
-$EndComp
-Wire Wire Line
-	3100 2950 3200 2950
-Wire Wire Line
-	3200 2950 3200 3050
-$Comp
-L power:GND #PWR02
+P 3200 3150
+F 0 "#PWR04" H 3200 2900 50  0001 C CNN
+F 1 "GND" H 3205 2977 50  0000 C CNN
+F 2 "" H 3200 3150 50  0001 C CNN
+F 3 "" H 3200 3150 50  0001 C CNN
+	1    3200 3150
+	1    0    0    -1
+$EndComp
+Wire Wire Line
+	3100 3050 3200 3050
+Wire Wire Line
+	3200 3050 3200 3150
+$Comp
+L power:GND #PWR01
 U 1 1 5CE49B9B
-P 2000 3050
-F 0 "#PWR02" H 2000 2800 50  0001 C CNN
-F 1 "GND" H 2005 2877 50  0000 C CNN
-F 2 "" H 2000 3050 50  0001 C CNN
-F 3 "" H 2000 3050 50  0001 C CNN
-	1    2000 3050
-	1    0    0    -1
-$EndComp
-Wire Wire Line
-	2000 3050 2000 2950
-Wire Wire Line
-	2000 2950 2100 2950
+P 2000 3150
+F 0 "#PWR01" H 2000 2900 50  0001 C CNN
+F 1 "GND" H 2005 2977 50  0000 C CNN
+F 2 "" H 2000 3150 50  0001 C CNN
+F 3 "" H 2000 3150 50  0001 C CNN
+	1    2000 3150
+	1    0    0    -1
+$EndComp
+Wire Wire Line
+	2000 3150 2000 3050
+Wire Wire Line
+	2000 3050 2100 3050
 Text GLabel 9250 1500 2    50   Output ~ 0
 V_RPI
@@
 $EndComp
 $Comp
-L power:+5V #PWR012
+L power:+5V #PWR09
 U 1 1 5CE7427A
 P 8400 2650
-F 0 "#PWR012" H 8400 2500 50  0001 C CNN
+F 0 "#PWR09" H 8400 2500 50  0001 C CNN
 F 1 "+5V" H 8415 2823 50  0000 C CNN
 F 2 "" H 8400 2650 50  0001 C CNN
@@
 $EndComp
 $Comp
-L power:GND #PWR015
+L power:GND #PWR012
 U 1 1 5CE74402
 P 8750 2700
-F 0 "#PWR015" H 8750 2450 50  0001 C CNN
+F 0 "#PWR012" H 8750 2450 50  0001 C CNN
 F 1 "GND" H 8750 2550 50  0000 C CNN
 F 2 "" H 8750 2700 50  0001 C CNN
@@
 $EndComp
 $Comp
-L power:GND #PWR014
+L power:GND #PWR011
 U 1 1 5CE760C6
 P 8750 2050
-F 0 "#PWR014" H 8750 1800 50  0001 C CNN
+F 0 "#PWR011" H 8750 1800 50  0001 C CNN
 F 1 "GND" H 8750 1900 50  0000 C CNN
 F 2 "" H 8750 2050 50  0001 C CNN
@@
 	5000 2950 5000 2850
 $Comp
-L power:GND #PWR08
+L power:GND #PWR05
 U 1 1 5CE8025B
 P 5400 3050
-F 0 "#PWR08" H 5400 2800 50  0001 C CNN
+F 0 "#PWR05" H 5400 2800 50  0001 C CNN
 F 1 "GND" H 5400 2900 50  0000 C CNN
 F 2 "" H 5400 3050 50  0001 C CNN
@@
 $EndComp
 $Comp
-L power:GND #PWR013
+L power:GND #PWR010
 U 1 1 5CED458D
 P 8550 4650
-F 0 "#PWR013" H 8550 4400 50  0001 C CNN
+F 0 "#PWR010" H 8550 4400 50  0001 C CNN
 F 1 "GND" H 8550 4500 50  0000 C CNN
 F 2 "" H 8550 4650 50  0001 C CNN
@@
 	-1   0    0    -1
 $EndComp
-Text GLabel 7600 5650 0    50   Input ~ 0
+Text GLabel 7350 5650 0    50   Input ~ 0
 CHG
 Wire Wire Line
@@
 Connection ~ 7850 5650
 Wire Wire Line
-	7850 5650 7600 5650
-Wire Wire Line
 	8200 5250 7850 5250
 Wire Wire Line
@@
 Wire Wire Line
 	9150 5900 9050 5900
-Text GLabel 7600 5250 0    50   Input ~ 0
+Text GLabel 7350 5250 0    50   Input ~ 0
 V_IN
-Wire Wire Line
-	7600 5250 7850 5250
 Connection ~ 7850 5250
 Wire Wire Line
@@
 Wire Wire Line
 	2900 3850 3000 3850
-Text GLabel 2000 2750 0    50   Input ~ 0
+Text GLabel 2000 2850 0    50   Input ~ 0
 V_BATT
 Wire Wire Line
-	2450 2550 2100 2550
-Wire Wire Line
-	2100 2550 2100 2750
-Connection ~ 2100 2750
-Wire Wire Line
-	2100 2750 2000 2750
+	2450 2650 2100 2650
+Wire Wire Line
+	2100 2650 2100 2850
+Connection ~ 2100 2850
+Wire Wire Line
+	2100 2850 2000 2850
 Text GLabel 9150 5900 2    50   Output ~ 0
 V_BATT
@@
 Text GLabel 9900 3200 2    50   Output ~ 0
 V_HDD
-Text GLabel 2550 1450 2    50   Input ~ 0
+Text GLabel 3400 1450 2    50   Input ~ 0
 V_HDD
 Wire Wire Line
 	9700 3200 9900 3200
 Wire Wire Line
-	2200 1350 2550 1350
-Wire Wire Line
-	2200 1450 2550 1450
+	2200 1350 2950 1350
+Wire Wire Line
+	2200 1450 2700 1450
+$Comp
+L Device:C C5
+U 1 1 5CEA3D6D
+P 8450 5250
+F 0 "C5" V 8300 5200 50  0000 R CNN
+F 1 "470nF" V 8300 5500 50  0000 R CNN
+F 2 "" H 8488 5100 50  0001 C CNN
+F 3 "~" H 8450 5250 50  0001 C CNN
+	1    8450 5250
+	0    1    1    0
+$EndComp
+$Comp
+L Device:C C1
+U 1 1 5CEC0215
+P 2700 1950
+F 0 "C1" H 2700 2050 50  0000 R CNN
+F 1 "220nF" H 2700 1850 50  0000 R CNN
+F 2 "" H 2738 1800 50  0001 C CNN
+F 3 "~" H 2700 1950 50  0001 C CNN
+	1    2700 1950
+	1    0    0    -1
+$EndComp
+$Comp
+L Device:C C2
+U 1 1 5CED4E79
+P 2950 1950
+F 0 "C2" H 2950 2050 50  0000 R CNN
+F 1 "220nF" H 2950 1850 50  0000 R CNN
+F 2 "" H 2988 1800 50  0001 C CNN
+F 3 "~" H 2950 1950 50  0001 C CNN
+	1    2950 1950
+	1    0    0    -1
+$EndComp
+Wire Wire Line
+	2300 2200 2700 2200
+Wire Wire Line
+	2700 2200 2700 2100
+Connection ~ 2300 2200
+Wire Wire Line
+	2300 2200 2300 1650
+Wire Wire Line
+	2700 2200 2950 2200
+Wire Wire Line
+	2950 2200 2950 2100
+Connection ~ 2700 2200
+Wire Wire Line
+	2700 1800 2700 1450
+Connection ~ 2700 1450
+Wire Wire Line
+	2700 1450 3400 1450
+Wire Wire Line
+	2950 1800 2950 1350
+Connection ~ 2950 1350
+Wire Wire Line
+	2950 1350 3200 1350
+Wire Wire Line
+	7350 5250 7850 5250
+Wire Wire Line
+	7350 5650 7850 5650
+$Comp
+L power:GND #PWR013
+U 1 1 5CEF6310
+P 8750 5300
+F 0 "#PWR013" H 8750 5050 50  0001 C CNN
+F 1 "GND" H 8750 5150 50  0000 C CNN
+F 2 "" H 8750 5300 50  0001 C CNN
+F 3 "" H 8750 5300 50  0001 C CNN
+	1    8750 5300
+	1    0    0    -1
+$EndComp
+Wire Wire Line
+	8200 5250 8300 5250
+Connection ~ 8200 5250
+Wire Wire Line
+	8600 5250 8750 5250
+Wire Wire Line
+	8750 5250 8750 5300
+$Comp
+L Device:CP C3
+U 1 1 5CF0005D
+P 3200 1950
+F 0 "C3" H 3000 2050 50  0000 L CNN
+F 1 "47µF/50V" H 2700 1850 50  0000 L CNN
+F 2 "" H 3238 1800 50  0001 C CNN
+F 3 "~" H 3200 1950 50  0001 C CNN
+	1    3200 1950
+	-1   0    0    -1
+$EndComp
+Wire Wire Line
+	3200 2100 3200 2200
+Wire Wire Line
+	3200 2200 2950 2200
+Connection ~ 2950 2200
+Wire Wire Line
+	3200 1800 3200 1350
+Connection ~ 3200 1350
+Wire Wire Line
+	3200 1350 3400 1350
 $EndSCHEMATC
