File: caravan/caravan-final.sch (KiCad schematic (older format))
At the start: 46 parts

Commit message: Updated caravan
Connections:
- wire segments 421 -> 422
Changed lines of the file:
@@
 Sheet 1 1
 Title "Autark-Schaltplan"
-Date "2021-11-10"
+Date "2022-04-17"
 Rev ""
 Comp ""
@@
 Wire Wire Line
 	6650 3900 6575 3900
-Text Notes 7000 7000 0    50   ~ 0
-Truma C4 Steuerung
+Text Notes 7000 7350 0    50   ~ 0
+Wasserpumpe/Toilette/Herd
 $Comp
 L Device:Fuse F?
@@
 Wire Wire Line
 	8300 7600 8250 7475
-Text Notes 7000 6825 0    50   ~ 0
+Text Notes 7000 6925 0    50   ~ 0
 Abwassertank-Heizung
 $Comp
@@
 Beleuchtung Kreis 3
 Text Notes 14750 4475 0    50   ~ 0
-Wasserpumpe/Toilette/Herd
+Truma C4 Steuerung
 Text Notes 14750 4675 0    50   ~ 0
 Kühlschrank
@@
 Kleiderschrank
 Wire Wire Line
-	4350 7600 4350 7525
+	4350 7600 4350 7475
 Connection ~ 4350 7600
 Wire Wire Line
@@
 	5725 7075 5900 7075
 Wire Wire Line
-	5900 7075 5900 7525
+	5900 7075 5900 7475
 Connection ~ 5750 6750
 Wire Wire Line
-	5925 7550 5925 7050
-Wire Wire Line
 	5925 7050 5750 7050
 Wire Wire Line
@@
 	6150 7050 5950 7050
 Wire Wire Line
-	5950 7050 5950 7550
-Wire Wire Line
 	6150 6750 6175 6750
 Wire Wire Line
@@
 	6175 7075 5975 7075
 Wire Wire Line
-	5975 7075 5975 7525
+	5975 7075 5975 7475
 Wire Wire Line
 	6150 6600 6200 6600
@@
 	6200 7100 6000 7100
 Wire Wire Line
-	6000 7100 6000 7500
-Wire Wire Line
-	6000 7500 6375 7500
-Wire Wire Line
-	6375 7500 6375 6450
-Wire Wire Line
-	6375 6450 6400 6450
-Wire Wire Line
-	5975 7525 6400 7525
-Wire Wire Line
-	6400 7525 6400 6775
-Wire Wire Line
-	6400 6775 6425 6775
-Wire Wire Line
-	6625 7450 6625 6975
-Wire Wire Line
-	6625 6975 6975 6975
+	6000 7100 6000 7450
+Wire Wire Line
+	6000 7450 6325 7450
+Wire Wire Line
+	6325 7450 6325 6450
+Wire Wire Line
+	6325 6450 6400 6450
+Wire Wire Line
+	5975 7475 6350 7475
+Wire Wire Line
+	6350 7475 6350 6875
+Wire Wire Line
+	6350 6875 6425 6875
+Wire Wire Line
+	6625 7450 6625 7325
+Wire Wire Line
+	6625 7325 6975 7325
 Wire Wire Line
 	6625 7450 8275 7450
@@
 	6600 7475 8250 7475
 Wire Wire Line
-	6600 6800 6975 6800
-Wire Wire Line
-	6600 6800 6600 7475
-Wire Wire Line
-	5950 7550 6425 7550
-Wire Wire Line
-	6425 7550 6425 6950
-Wire Wire Line
-	6425 6950 6450 6950
-Text Label 5900 7200 3    39   ~ 0
+	6600 6900 6975 6900
+Wire Wire Line
+	6600 6900 6600 7475
+Wire Wire Line
+	6425 7550 6425 7300
+Text Label 5900 7100 3    39   ~ 0
 5x1.5mm2
 Wire Wire Line
@@
 	6400 6450 6650 6450
 Wire Wire Line
-	6425 6775 6425 6800
-Connection ~ 6425 6775
-Wire Wire Line
-	6425 6775 6975 6775
-Wire Wire Line
-	6450 6950 6450 6975
-Connection ~ 6450 6950
-Wire Wire Line
-	6450 6950 6975 6950
-Text Label 6625 6775 0    39   ~ 0
+	6425 6875 6425 6900
+Connection ~ 6425 6875
+Wire Wire Line
+	6425 6875 6975 6875
+Text Label 6625 6875 0    39   ~ 0
 2x2.5mm2
-Text Label 6625 6950 0    39   ~ 0
+Text Label 6625 7300 0    39   ~ 0
 2x2.5mm2
 Wire Wire Line
@@
 	4825 3900 4825 6150
 Wire Wire Line
-	4575 5800 4575 5450
-Connection ~ 4575 5450
-Wire Wire Line
-	4575 5450 4625 5500
-Wire Wire Line
-	4625 5500 4625 5800
+	4575 5800 4575 5500
+Connection ~ 4575 5500
+Wire Wire Line
+	4575 5500 4625 5550
+Wire Wire Line
+	4625 5550 4625 5800
 Wire Wire Line
 	10350 7400 12525 7400
@@
 	10375 5800 10375 7375
 Connection ~ 12525 7250
-Wire Wire Line
-	3575 3950 3575 5450
 Text Label 3125 5800 0    50   ~ 0
 2x4mm2
@@
 Wire Wire Line
 	1775 5725 2125 5725
-Wire Wire Line
-	3575 5450 4575 5450
 Wire Wire Line
 	3600 3900 3300 3900
@@
 	4325 3950 4325 5275
 Wire Wire Line
-	4350 7525 5900 7525
-Wire Wire Line
-	4525 7550 5925 7550
+	4350 7475 5900 7475
 Wire Wire Line
 	5400 3900 5400 8325
@@
 	5300 8325 5300 8425
 Wire Wire Line
-	4575 5350 4575 5450
+	4575 5350 4575 5500
 Wire Wire Line
 	4675 4050 4675 4300
@@
 Wire Wire Line
 	4675 5825 4675 5425
-Wire Wire Line
-	4625 5375 4575 5450
-Wire Wire Line
-	5250 5375 4625 5375
 Wire Wire Line
 	2150 5075 4950 5075
@@
 Text Notes 4950 4750 0    39   ~ 0
 Transistor
-Text Notes 3200 2875 0    50   ~ 0
-Notizen zum Votronic Ladewandler:\nDas Relais unterbindet den Rückladezweig und verhindert damit das\nEinschalten vom ATC ohne Zugfahrzeug.\nDer Transistor aktiviert den Ladevorgang nur wenn ATC-Schaltplus UND \nZugfahrzeug-D+ beide aktiv sind. Damit wird der Ladevorgang unterbrochen,\nwenn der Motor aus oder die ATC-Bremse aktiv ist. \nDie Ideale Diode ermöglicht das gleichzeitige Nutzen der Shaltplus- und \nDauerplus-Leitungen zum Laden der Batterie. Dies ermöglicht die\noptimale Nutzung des Leitungsquerschnitts.
+Text Notes 3050 2700 0    50   ~ 0
+Notizen zum Votronic Ladewandler:\nDas Relais unterbindet den Rückladezweig und verhindert damit das\nEinschalten vom ATC ohne Zugfahrzeug.\nDer Transistor aktiviert den Ladevorgang nur wenn ATC-Schaltplus UND \nZugfahrzeug-D+ beide aktiv sind. Damit wird der Ladevorgang unterbrochen,\nwenn der Motor aus oder die ATC-Bremse aktiv ist. \nDie Ideale Diode ermöglicht das gleichzeitige Nutzen der Shaltplus- und \nDauerplus-Leitungen zum Laden der Batterie. Dies ermöglicht die\noptimale Nutzung des Leitungsquerschnitts.\nDer Ladewandler kann mittels eines Schalters deaktiviert werden.
 Wire Wire Line
 	4950 5075 4975 5075
@@
 Text Label 4825 4900 1    50   ~ 0
 4mm2|6mm2
+Wire Wire Line
+	4525 7550 6425 7550
+Wire Wire Line
+	6425 7300 6975 7300
+Wire Wire Line
+	3575 3950 3575 5375
+Wire Wire Line
+	3575 5375 4500 5375
+Wire Wire Line
+	4500 7450 5925 7450
+Wire Wire Line
+	5925 7450 5925 7050
+Wire Wire Line
+	5950 7050 5950 7425
+Wire Wire Line
+	5950 7425 4525 7425
+Wire Wire Line
+	4500 5375 4500 7450
+Connection ~ 4500 5375
+Wire Wire Line
+	4500 5375 5250 5375
+Wire Wire Line
+	4525 5550 4575 5500
+Wire Wire Line
+	4525 5550 4525 7425
 $EndSCHEMATC

Commit message: caravan: Add fuses for Votronic booster and Victron MPPT
Parts:
- added F?: 20A, symbol Device:Fuse
- added F?: 30A Maxi, symbol Device:Fuse
- added F?: Reserve Maxi, symbol Device:Fuse
- F?: value 30A -> 30A Maxi
- F?: value 50A -> 50A MIDI
- F? (x2): value 25A -> 25A Maxi
Connections:
- net labels removed: 4mm2|6mm2
- wire segments 422 -> 423
Other:
- note added: "Lade-Wandler"
- note added: "Lade-Wandler (Nr. 3321)"
- note added: "Notizen zum Votronic Lade-Wandler:\nDas Relais unterbindet den Rückladezweig und verhindert damit das\nEinschalten vom ATC ohne Zugfahrzeug.\nDer Transistor aktiviert den Ladevorgang nur wenn ATC-Schaltplus UND \nZugfahrzeug-D+ beide aktiv sind. Damit wird der Ladevorgang unterbrochen,\nwenn der Motor aus oder die ATC-Bremse aktiv ist. \nDie Ideale Diode ermöglicht das gleichzeitige Nutzen der Sh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"
- note added: "Solarladeregler"
- note removed: "Ladewandler (Nr. 3321)"
- note removed: "Notizen zum Votronic Ladewandler:\nDas Relais unterbindet den Rückladezweig und verhindert damit das\nEinschalten vom ATC ohne Zugfahrzeug.\nDer Transistor aktiviert den Ladevorgang nur wenn ATC-Schaltplus UND \nZugfahrzeug-D+ beide aktiv sind. Damit wird der Ladevorgang unterbrochen,\nwenn der Motor aus oder die ATC-Bremse aktiv ist. \nDie Ideale Diode ermöglicht das gleichzeitige Nutzen der Sha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"
Changed lines of the file:
@@
 Sheet 1 1
 Title "Autark-Schaltplan"
-Date "2022-04-17"
+Date "2022-04-26"
 Rev ""
 Comp ""
@@
 Wire Wire Line
 	12475 4850 12475 4900
-Wire Wire Line
-	4175 7925 4175 7600
 Text Label 13050 3300 0    50   ~ 0
 PE
@@
 	11200 6575 12525 6575
 Wire Wire Line
-	8550 6150 11425 6150
-Wire Wire Line
-	11425 6150 11425 5150
-Wire Wire Line
-	11400 6125 11400 5125
+	11400 6025 11400 5125
 $Comp
 L power:Earth #PWR?
@@
 Wire Wire Line
 	10025 3075 10025 2875
-Wire Wire Line
-	4875 6100 4875 6075
-Wire Wire Line
-	4875 6100 8550 6100
-Wire Wire Line
-	4150 6100 4150 7575
 Wire Wire Line
 	9800 3075 9800 4000
@@
 P 4650 9250
 F 0 "F?" H 4710 9296 50  0001 L CNN
-F 1 "50A" V 4575 9175 50  0000 L CNN
+F 1 "50A MIDI" V 4575 9075 50  0000 L CNN
 F 2 "" V 4580 9250 50  0001 C CNN
 F 3 "~" H 4650 9250 50  0001 C CNN
@@
 L Device:Fuse F?
 U 1 1 6048F6FE
-P 4175 8075
-F 0 "F?" H 4235 8121 50  0001 L CNN
-F 1 "30A" V 4100 8000 50  0000 L CNN
-F 2 "" V 4105 8075 50  0001 C CNN
-F 3 "~" H 4175 8075 50  0001 C CNN
-	1    4175 8075
-	1    0    0    -1
-$EndComp
-Wire Wire Line
-	4200 7575 4175 7600
-Connection ~ 4175 7600
-Wire Wire Line
-	4175 7600 4175 6125
-Wire Wire Line
-	4150 7575 4175 7600
-Wire Wire Line
-	8550 6150 8550 7600
+P 4000 8075
+F 0 "F?" H 4060 8121 50  0001 L CNN
+F 1 "30A Maxi" V 3925 7900 50  0000 L CNN
+F 2 "" V 3930 8075 50  0001 C CNN
+F 3 "~" H 4000 8075 50  0001 C CNN
+	1    4000 8075
+	1    0    0    -1
+$EndComp
 Wire Wire Line
 	8525 7575 8550 7600
@@
 Wire Wire Line
 	8275 7450 8300 7600
-Text Label 4150 7050 3    50   ~ 0
-Wago221-615
 Wire Wire Line
 	8550 9250 8550 9175
@@
 Text Label 5775 9200 0    39   ~ 0
 Busbar
-Text Label 4175 8450 1    39   ~ 0
-6mm2
-Text Label 4175 7875 1    39   ~ 0
+Text Label 4175 8475 1    39   ~ 0
+2.5mm2
+Text Label 4000 7900 1    39   ~ 0
 6mm2
 Text Label 8525 7050 3    50   ~ 0
@@
 Text Label 4425 9350 0    50   ~ 0
 M5
-Text Label 3975 8600 0    50   ~ 0
+Text Label 3975 8650 0    50   ~ 0
 M10
-Text Label 3975 8950 0    50   ~ 0
+Text Label 3975 8900 0    50   ~ 0
 M10
 Text Label 8575 9175 0    50   ~ 0
@@
 Wire Wire Line
 	9850 4050 8725 4050
-Wire Wire Line
-	4175 8225 4175 8550
-Text Label 4025 7975 0    50   ~ 0
-M5
-Text Label 4025 8250 0    50   ~ 0
-M5
-Wire Wire Line
-	4525 8225 4525 8550
 Wire Wire Line
 	4200 8525 4175 8550
@@
 Connection ~ 4175 8550
 Wire Wire Line
-	4175 8550 4525 8550
+	4175 8550 4150 8575
 Wire Wire Line
 	4200 8525 4350 8525
@@
 Wire Wire Line
 	8300 8175 8300 7600
-Text Label 9775 6125 0    50   ~ 0
+Text Label 9775 6025 0    50   ~ 0
 2x6mm2
 $Comp
@@
 Wire Wire Line
 	2150 4600 2150 5075
-Wire Wire Line
-	4800 6125 4800 6150
-Wire Wire Line
-	4800 6150 4200 6150
-Wire Wire Line
-	4200 6150 4200 7575
-Wire Wire Line
-	4850 6100 4775 6100
-Wire Wire Line
-	4775 6100 4775 6125
-Wire Wire Line
-	4775 6125 4175 6125
-Wire Wire Line
-	4875 6075 4750 6075
-Wire Wire Line
-	4750 6075 4750 6100
-Wire Wire Line
-	4750 6100 4150 6100
-Wire Wire Line
-	8525 6150 8525 7575
 Wire Wire Line
 	2175 5050 2150 5075
@@
 	14625 5150 14650 5150
 Wire Wire Line
-	8525 6150 4825 6150
-Wire Wire Line
 	4700 3900 4825 3900
 Wire Wire Line
@@
 	8575 3900 8575 7575
 Wire Wire Line
-	4800 6125 11400 6125
-Wire Wire Line
-	8550 3900 8550 6100
-Wire Wire Line
 	6650 3900 6650 6450
 Wire Wire Line
 	6675 3900 6675 6450
 Wire Wire Line
-	4825 3900 4825 6150
+	4825 3900 4825 5900
 Wire Wire Line
 	4575 5800 4575 5500
@@
 P 2375 5200
 F 0 "F?" H 2435 5246 50  0001 L CNN
-F 1 "25A" V 2300 5125 50  0000 L CNN
+F 1 "25A Maxi" V 2300 5025 50  0000 L CNN
 F 2 "" V 2305 5200 50  0001 C CNN
 F 3 "~" H 2375 5200 50  0001 C CNN
@@
 P 1975 6125
 F 0 "F?" H 2035 6171 50  0001 L CNN
-F 1 "25A" V 1900 6050 50  0000 L CNN
+F 1 "25A Maxi" V 1900 5950 50  0000 L CNN
 F 2 "" V 1905 6125 50  0001 C CNN
 F 3 "~" H 1975 6125 50  0001 C CNN
@@
 	2625 5200 2625 5100
 Text Label 8550 4900 1    50   ~ 0
-2x6mm2
+2x4mm2
 Wire Wire Line
 	2625 5250 4425 5250
@@
 Transistor
 Text Notes 3050 2700 0    50   ~ 0
-Notizen zum Votronic Ladewandler:\nDas Relais unterbindet den Rückladezweig und verhindert damit das\nEinschalten vom ATC ohne Zugfahrzeug.\nDer Transistor aktiviert den Ladevorgang nur wenn ATC-Schaltplus UND \nZugfahrzeug-D+ beide aktiv sind. Damit wird der Ladevorgang unterbrochen,\nwenn der Motor aus oder die ATC-Bremse aktiv ist. \nDie Ideale Diode ermöglicht das gleichzeitige Nutzen der Shaltplus- und \nDauerplus-Leitungen zum Laden der Batterie. Dies ermöglicht die\noptimale Nutzung des Leitungsquerschnitts.\nDer Ladewandler kann mittels eines Schalters deaktiviert werden.
+Notizen zum Votronic Lade-Wandler:\nDas Relais unterbindet den Rückladezweig und verhindert damit das\nEinschalten vom ATC ohne Zugfahrzeug.\nDer Transistor aktiviert den Ladevorgang nur wenn ATC-Schaltplus UND \nZugfahrzeug-D+ beide aktiv sind. Damit wird der Ladevorgang unterbrochen,\nwenn der Motor aus oder die ATC-Bremse aktiv ist. \nDie Ideale Diode ermöglicht das gleichzeitige Nutzen der Shaltplus- und \nDauerplus-Leitungen zum Laden der Batterie. Dies ermöglicht die\noptimale Nutzung des Leitungsquerschnitts.\nDer Ladewandler kann mittels eines Schalters deaktiviert werden.
 Wire Wire Line
 	4950 5075 4975 5075
@@
 	4000 4175 4850 4175
 Wire Wire Line
-	4850 4175 4850 6100
+	4850 4175 4850 5925
 Wire Wire Line
 	4150 3250 4150 4150
@@
 $EndComp
 Text Notes 4425 3350 0    50   ~ 0
-Ladewandler (Nr. 3321)
+Lade-Wandler (Nr. 3321)
 Text Notes 3650 3900 0    50   ~ 0
 Relais
@@
 2x2.5mm2
 Text Label 4825 4900 1    50   ~ 0
-4mm2|6mm2
+2x4mm2
 Wire Wire Line
 	4525 7550 6425 7550
@@
 Wire Wire Line
 	4525 5550 4525 7425
+$Comp
+L Device:Fuse F?
+U 1 1 626DA299
+P 4175 8075
+F 0 "F?" H 4235 8121 50  0001 L CNN
+F 1 "20A" V 4100 8000 50  0000 L CNN
+F 2 "" V 4105 8075 50  0001 C CNN
+F 3 "~" H 4175 8075 50  0001 C CNN
+	1    4175 8075
+	1    0    0    -1
+$EndComp
+$Comp
+L Device:Fuse F?
+U 1 1 626DA689
+P 3825 8075
+F 0 "F?" H 3885 8121 50  0001 L CNN
+F 1 "30A Maxi" V 3750 7900 50  0000 L CNN
+F 2 "" V 3755 8075 50  0001 C CNN
+F 3 "~" H 3825 8075 50  0001 C CNN
+	1    3825 8075
+	1    0    0    -1
+$EndComp
+Wire Wire Line
+	3825 8550 3825 8225
+Wire Wire Line
+	3825 8550 4175 8550
+Wire Wire Line
+	3825 7925 3825 5925
+Wire Wire Line
+	3825 5925 4850 5925
+Wire Wire Line
+	4825 5900 4875 5900
+Wire Wire Line
+	4875 5900 4875 5925
+Wire Wire Line
+	4875 5925 8525 5925
+Wire Wire Line
+	8525 5925 8525 7575
+Text Label 4000 8450 1    39   ~ 0
+4mm2
+Text Label 3825 8450 1    39   ~ 0
+4mm2
+Text Label 4175 7900 1    39   ~ 0
+4mm2
+Text Label 3825 7900 1    39   ~ 0
+4mm2
+Wire Wire Line
+	3675 8575 3675 8225
+Wire Wire Line
+	4175 8550 4525 8550
+Wire Wire Line
+	4525 8550 4525 8225
+Text Label 3675 8275 3    39   ~ 0
+4mm2
+Wire Wire Line
+	4000 6025 4000 7925
+Wire Wire Line
+	4175 8225 4175 8550
+Wire Wire Line
+	4175 6125 4175 7925
+Wire Wire Line
+	4175 6125 8350 6125
+Wire Wire Line
+	4000 6025 11400 6025
+Wire Wire Line
+	8550 6050 11425 6050
+Wire Wire Line
+	11425 6050 11425 5150
+Wire Wire Line
+	8550 6050 8550 7600
+Wire Wire Line
+	8350 6125 8350 5700
+Wire Wire Line
+	8350 5700 8550 5700
+Wire Wire Line
+	8550 5700 8550 3900
+Wire Wire Line
+	4000 8225 4000 8525
+Wire Wire Line
+	4000 8525 4150 8525
+Wire Wire Line
+	4150 8525 4175 8550
+Wire Wire Line
+	4150 8575 3675 8575
+Text Notes 3825 7675 1    50   ~ 0
+Lade-Wandler
+Text Notes 4175 7675 1    50   ~ 0
+Solarladeregler
+Text Notes 4000 7675 1    50   ~ 0
+12V Verteiler
+$Comp
+L Device:Fuse F?
+U 1 1 62BF37F1
+P 3675 8075
+F 0 "F?" H 3735 8121 50  0001 L CNN
+F 1 "Reserve Maxi" V 3600 7875 50  0000 L CNN
+F 2 "" V 3605 8075 50  0001 C CNN
+F 3 "~" H 3675 8075 50  0001 C CNN
+	1    3675 8075
+	1    0    0    -1
+$EndComp
 $EndSCHEMATC

Commit message: caravan: Maxi fuse for Victorn MPPT
Parts:
- F?: value 20A -> 30A Maxi
- F?: value Reserve Maxi -> Reserve
Connections:
- wire segments 423 -> 421
Other:
- note added: "Ladewandler"
- note added: "Ladewandler (Nr. 3321)"
- note added: "Notizen zum Votronic Ladewandler:\nDas Relais unterbindet den Rückladezweig und verhindert damit das\nEinschalten vom ATC ohne Zugfahrzeug.\nDer Transistor aktiviert den Ladevorgang nur wenn ATC-Schaltplus UND \nZugfahrzeug-D+ beide aktiv sind. Damit wird der Ladevorgang unterbrochen,\nwenn der Motor aus oder die ATC-Bremse aktiv ist. \nDie Ideale Diode ermöglicht das gleichzeitige Nutzen der Sha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"
- note removed: "Lade-Wandler"
- note removed: "Lade-Wandler (Nr. 3321)"
- note removed: "Notizen zum Votronic Lade-Wandler:\nDas Relais unterbindet den Rückladezweig und verhindert damit das\nEinschalten vom ATC ohne Zugfahrzeug.\nDer Transistor aktiviert den Ladevorgang nur wenn ATC-Schaltplus UND \nZugfahrzeug-D+ beide aktiv sind. Damit wird der Ladevorgang unterbrochen,\nwenn der Motor aus oder die ATC-Bremse aktiv ist. \nDie Ideale Diode ermöglicht das gleichzeitige Nutzen der Sh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"
Changed lines of the file:
@@
 	11200 6575 12525 6575
 Wire Wire Line
-	11400 6025 11400 5125
+	8550 6150 11425 6150
+Wire Wire Line
+	11425 6150 11425 5150
+Wire Wire Line
+	11400 6125 11400 5125
 $Comp
 L power:Earth #PWR?
@@
 L Device:Fuse F?
 U 1 1 6048F6FE
-P 4000 8075
-F 0 "F?" H 4060 8121 50  0001 L CNN
-F 1 "30A Maxi" V 3925 7900 50  0000 L CNN
-F 2 "" V 3930 8075 50  0001 C CNN
-F 3 "~" H 4000 8075 50  0001 C CNN
-	1    4000 8075
-	1    0    0    -1
-$EndComp
+P 4175 8075
+F 0 "F?" H 4235 8121 50  0001 L CNN
+F 1 "30A Maxi" V 4100 7900 50  0000 L CNN
+F 2 "" V 4105 8075 50  0001 C CNN
+F 3 "~" H 4175 8075 50  0001 C CNN
+	1    4175 8075
+	1    0    0    -1
+$EndComp
+Wire Wire Line
+	8550 6150 8550 7600
 Wire Wire Line
 	8525 7575 8550 7600
@@
 Text Label 5775 9200 0    39   ~ 0
 Busbar
-Text Label 4175 8475 1    39   ~ 0
-2.5mm2
-Text Label 4000 7900 1    39   ~ 0
+Text Label 4175 8450 1    39   ~ 0
+4mm2
+Text Label 4175 7875 1    39   ~ 0
 6mm2
 Text Label 8525 7050 3    50   ~ 0
@@
 	9850 4050 8725 4050
 Wire Wire Line
+	4175 8225 4175 8550
+Wire Wire Line
 	4200 8525 4175 8550
 Text Label 4350 8250 3    39   ~ 0
@@
 Connection ~ 4175 8550
 Wire Wire Line
-	4175 8550 4150 8575
+	4175 8550 4200 8575
 Wire Wire Line
 	4200 8525 4350 8525
@@
 Wire Wire Line
 	8300 8175 8300 7600
-Text Label 9775 6025 0    50   ~ 0
+Text Label 9775 6125 0    50   ~ 0
 2x6mm2
 $Comp
@@
 	8575 3900 8575 7575
 Wire Wire Line
+	8550 3900 8550 6025
+Wire Wire Line
 	6650 3900 6650 6450
 Wire Wire Line
@@
 Transistor
 Text Notes 3050 2700 0    50   ~ 0
-Notizen zum Votronic Lade-Wandler:\nDas Relais unterbindet den Rückladezweig und verhindert damit das\nEinschalten vom ATC ohne Zugfahrzeug.\nDer Transistor aktiviert den Ladevorgang nur wenn ATC-Schaltplus UND \nZugfahrzeug-D+ beide aktiv sind. Damit wird der Ladevorgang unterbrochen,\nwenn der Motor aus oder die ATC-Bremse aktiv ist. \nDie Ideale Diode ermöglicht das gleichzeitige Nutzen der Shaltplus- und \nDauerplus-Leitungen zum Laden der Batterie. Dies ermöglicht die\noptimale Nutzung des Leitungsquerschnitts.\nDer Ladewandler kann mittels eines Schalters deaktiviert werden.
+Notizen zum Votronic Ladewandler:\nDas Relais unterbindet den Rückladezweig und verhindert damit das\nEinschalten vom ATC ohne Zugfahrzeug.\nDer Transistor aktiviert den Ladevorgang nur wenn ATC-Schaltplus UND \nZugfahrzeug-D+ beide aktiv sind. Damit wird der Ladevorgang unterbrochen,\nwenn der Motor aus oder die ATC-Bremse aktiv ist. \nDie Ideale Diode ermöglicht das gleichzeitige Nutzen der Shaltplus- und \nDauerplus-Leitungen zum Laden der Batterie. Dies ermöglicht die\noptimale Nutzung des Leitungsquerschnitts.\nDer Ladewandler kann mittels eines Schalters deaktiviert werden.
 Wire Wire Line
 	4950 5075 4975 5075
@@
 $EndComp
 Text Notes 4425 3350 0    50   ~ 0
-Lade-Wandler (Nr. 3321)
+Ladewandler (Nr. 3321)
 Text Notes 3650 3900 0    50   ~ 0
 Relais
@@
 L Device:Fuse F?
 U 1 1 626DA299
-P 4175 8075
-F 0 "F?" H 4235 8121 50  0001 L CNN
-F 1 "20A" V 4100 8000 50  0000 L CNN
-F 2 "" V 4105 8075 50  0001 C CNN
-F 3 "~" H 4175 8075 50  0001 C CNN
-	1    4175 8075
+P 4000 8075
+F 0 "F?" H 4060 8121 50  0001 L CNN
+F 1 "30A Maxi" V 3925 7900 50  0000 L CNN
+F 2 "" V 3930 8075 50  0001 C CNN
+F 3 "~" H 4000 8075 50  0001 C CNN
+	1    4000 8075
 	1    0    0    -1
 $EndComp
@@
 	3825 8550 3825 8225
 Wire Wire Line
+	4000 8225 4000 8525
+Wire Wire Line
+	4000 8525 4150 8525
+Wire Wire Line
+	4175 8550 4150 8525
+Wire Wire Line
 	3825 8550 4175 8550
 Wire Wire Line
+	4000 6025 8550 6025
+Wire Wire Line
+	4000 6025 4000 7925
+Wire Wire Line
 	3825 7925 3825 5925
 Wire Wire Line
 	3825 5925 4850 5925
+Wire Wire Line
+	4175 6125 11400 6125
 Wire Wire Line
 	4825 5900 4875 5900
@@
 Text Label 3825 8450 1    39   ~ 0
 4mm2
-Text Label 4175 7900 1    39   ~ 0
+Text Label 4000 7875 1    39   ~ 0
 4mm2
-Text Label 3825 7900 1    39   ~ 0
+Text Label 3825 7875 1    39   ~ 0
 4mm2
-Wire Wire Line
-	3675 8575 3675 8225
+$Comp
+L Device:Fuse F?
+U 1 1 62BF37F1
+P 4700 8075
+F 0 "F?" H 4760 8121 50  0001 L CNN
+F 1 "Reserve" V 4625 7925 50  0000 L CNN
+F 2 "" V 4630 8075 50  0001 C CNN
+F 3 "~" H 4700 8075 50  0001 C CNN
+	1    4700 8075
+	1    0    0    -1
+$EndComp
+Wire Wire Line
+	4200 8575 4700 8575
+Wire Wire Line
+	4700 8575 4700 8225
 Wire Wire Line
 	4175 8550 4525 8550
 Wire Wire Line
 	4525 8550 4525 8225
-Text Label 3675 8275 3    39   ~ 0
+Text Label 4700 8250 3    39   ~ 0
 4mm2
 Wire Wire Line
-	4000 6025 4000 7925
-Wire Wire Line
-	4175 8225 4175 8550
-Wire Wire Line
 	4175 6125 4175 7925
-Wire Wire Line
-	4175 6125 8350 6125
-Wire Wire Line
-	4000 6025 11400 6025
-Wire Wire Line
-	8550 6050 11425 6050
-Wire Wire Line
-	11425 6050 11425 5150
-Wire Wire Line
-	8550 6050 8550 7600
-Wire Wire Line
-	8350 6125 8350 5700
-Wire Wire Line
-	8350 5700 8550 5700
-Wire Wire Line
-	8550 5700 8550 3900
-Wire Wire Line
-	4000 8225 4000 8525
-Wire Wire Line
-	4000 8525 4150 8525
-Wire Wire Line
-	4150 8525 4175 8550
-Wire Wire Line
-	4150 8575 3675 8575
-Text Notes 3825 7675 1    50   ~ 0
-Lade-Wandler
-Text Notes 4175 7675 1    50   ~ 0
+Text Notes 3825 7625 1    50   ~ 0
+Ladewandler
+Text Notes 4000 7625 1    50   ~ 0
 Solarladeregler
-Text Notes 4000 7675 1    50   ~ 0
+Text Notes 4175 7625 1    50   ~ 0
 12V Verteiler
-$Comp
-L Device:Fuse F?
-U 1 1 62BF37F1
-P 3675 8075
-F 0 "F?" H 3735 8121 50  0001 L CNN
-F 1 "Reserve Maxi" V 3600 7875 50  0000 L CNN
-F 2 "" V 3605 8075 50  0001 C CNN
-F 3 "~" H 3675 8075 50  0001 C CNN
-	1    3675 8075
-	1    0    0    -1
-$EndComp
 $EndSCHEMATC
