File: caravan/caravan.kicad_sch (KiCad schematic)
At the start: 51 parts

Commit message: Updated caravan schematic
Parts:
- removed F?: 1A, symbol Device:Fuse
- added F?: 50A MIDI, symbol Device:Fuse
- added U?: Victron Phoenix 12|500, symbol microfarad-de:Victron_Inverter_Phoenix
- U?: value BMS 100A -> JBD BMS 120A
Connections:
- net Earth: now also K?.85, Q?.1 (C), F?.1, U?. (Remote_2); no longer F?.1, F?.2, F?.2, F?.2, F?.2
- net at SW?.2 (B): now also U?. (Remote_2)
- new net: F?.1, F?.2, F?.2, F?.2, F?.2, F?.2
- new net: SW?.1 (A), U?. (Remote_2)
Other:
- note added: "Inverter"
- note added: "Wechselrichter"
- note removed: "Booster"
