File: smart-pump/smart-pump.sch (KiCad schematic (older format))
At the start: 19 parts, among them J1 Screw_Terminal_01x04, Q1 BC337, Q2 IRF5305, SW1 SW_SPST, U1 AZ1117-5.0, U2 Arduino_Pro_Mini

Commit message: Updated smart-pump
Parts:
- removed U1: AZ1117-5.0, symbol Regulator_Linear:AZ1117-5.0
- added U1: AMS1117-5.0, Package_TO_SOT_SMD:SOT-223-3_TabPin2, symbol Regulator_Linear:AMS1117-5.0
Connections:
- net +12V: now also U1.3 (VI)
- net +5V: now also U1.2 (VO)
- net GND: now also U1.1 (GND)
Changed lines of the file:
@@
-$EndComp
-$Comp
-L Regulator_Linear:AZ1117-5.0 U1
-U 1 1 624A95B3
-P 1725 1325
-F 0 "U1" H 1725 1567 50  0000 C CNN
-F 1 "AZ1117-5.0" H 1725 1476 50  0000 C CNN
-F 2 "" H 1725 1575 50  0001 C CIN
-F 3 "https://www.diodes.com/assets/Datasheets/AZ1117.pdf" H 1725 1325 50  0001 C CNN
-	1    1725 1325
-	1    0    0    -1
 $EndComp
 $Comp
@@
 Wire Wire Line
 	3725 1225 3725 1525
+$Comp
+L Regulator_Linear:AMS1117-5.0 U1
+U 1 1 6259A42F
+P 1725 1325
+F 0 "U1" H 1725 1567 50  0000 C CNN
+F 1 "AMS1117-5.0" H 1725 1476 50  0000 C CNN
+F 2 "Package_TO_SOT_SMD:SOT-223-3_TabPin2" H 1725 1525 50  0001 C CNN
+F 3 "http://www.advanced-monolithic.com/pdf/ds1117.pdf" H 1825 1075 50  0001 C CNN
+	1    1725 1325
+	1    0    0    -1
+$EndComp
 $EndSCHEMATC

Commit message: Updated smart-pump
Parts:
- added R1: 13kΩ, symbol Device:R
- added R2: 1kΩ, symbol Device:R
- renumbered R8 to R10, R1 to R3, R2 to R4, R3 to R5, R4 to R6, R5 to R7, R6 to R8, R7 to R9
Connections:
- net +12V: now also R1.1
- net GND: now also R2.2
- net at U2.20 (A3): now also R1.2, R2.1
Other:
- moved on the sheet: C3, D1, D2, Q1, Q2, R10, R3, R4, R5, R6, R7, R8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

Commit message: Updated smart-pump
Parts:
- R1: value 13kΩ -> 12kΩ
Changed lines of the file:
@@
 Sheet 1 1
 Title "Smart Water Pump"
-Date "2022-04-11"
+Date "2022-04-12"
 Rev ""
 Comp "µF"
@@
 P 3375 1425
 F 0 "R1" H 3445 1471 50  0000 L CNN
-F 1 "13kΩ" H 3445 1380 50  0000 L CNN
+F 1 "12kΩ" H 3445 1380 50  0000 L CNN
 F 2 "" V 3305 1425 50  0001 C CNN
 F 3 "~" H 3375 1425 50  0001 C CNN

Commit message: Updated smart pump
Parts:
- removed J1: Screw_Terminal_01x04, symbol Connector:Screw_Terminal_01x04
- removed Q1: BC337, Package_TO_SOT_THT:TO-92_Inline, symbol Transistor_BJT:BC337
- removed Q2: IRF5305, symbol Device:Q_PMOS_GDS
- removed R2: 1kΩ, symbol Device:R
- removed R5, R6: 10kΩ, symbol Device:R
- added C3: 100nF, symbol Device:C
- added J1: Screw_Terminal_01x03, symbol Connector:Screw_Terminal_01x03
- added J2: Screw_Terminal_01x02, symbol Connector:Screw_Terminal_01x02
- added Q1: IRF8721PBF, Package_SO:SOIC-8_3.9x4.9mm_P1.27mm, symbol Transistor_FET:IRF8721PBF-1
- R1: value 12kΩ -> 1MΩ
- renumbered C3 to C4, R3 to R2, R4 to R3, R7 to R4, R8 to R5, R9 to R6, R10 to R7
Connections:
- net M+ is gone; now on net +12V: D2.1 (K)
- net +12V: now also J1.3 (Pin_3), J2.2 (Pin_2); no longer R1.1
- net +5V: now also R1.1
- net GND: now also C3.2, J1.1 (Pin_1)
- net M-: now also J2.1 (Pin_1), Q1.5 (D), Q1.6 (D), Q1.7 (D), Q1.8 (D); no longer R3.1, R4.1, R5.1, R6.1, R7.1
- net at U2.12 (9*): now also Q1.4 (G)
- net LEVEL: now reaches R1.2, U2.20 (A3)
- net LEVEL: now also C3.1, J1.2 (Pin_2)
- new net: Q1.1 (S), Q1.2 (S), Q1.3 (S), R3.1, R4.1, R5.1, R6.1, R7.1
Other:
- moved on the sheet: C1, C2, C4, D1, D2, R1, R2, R3, R4, R5, R6, R7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

Commit message: Updated smart-pump
Parts:
- removed C3: 100nF, symbol Device:C
- added R2: 330kΩ, symbol Device:R
- renumbered C4 to C3, R2 to R3, R3 to R4, R4 to R5, R5 to R6, R6 to R7, R7 to R8
Connections:
- net GND: now also R2.2
- net LEVEL: now also R2.1
Changed lines of the file:
@@
 Sheet 1 1
 Title "Smart Water Pump"
-Date "2022-04-23"
+Date "2022-04-24"
 Rev ""
 Comp "µF"
@@
 $EndComp
 $Comp
-L Device:C C4
+L Device:C C3
 U 1 1 624A13A7
 P 4325 3200
-F 0 "C4" H 4440 3246 50  0000 L CNN
+F 0 "C3" H 4440 3246 50  0000 L CNN
 F 1 "100nF" H 4440 3155 50  0000 L CNN
 F 2 "" H 4363 3050 50  0001 C CNN
@@
 	1800 2225 1800 2200
 $Comp
-L Device:R R4
+L Device:R R5
 U 1 1 624BB180
 P 5900 3200
-F 0 "R4" V 5800 3000 50  0000 L CNN
+F 0 "R5" V 5800 3000 50  0000 L CNN
 F 1 "1Ω/1W" V 5800 3150 50  0000 L CNN
 F 2 "" V 5830 3200 50  0001 C CNN
@@
 	1800 2425 1800 2450
 $Comp
-L Device:R R5
+L Device:R R6
 U 1 1 624C399C
 P 6100 3200
-F 0 "R5" V 6000 3000 50  0000 L CNN
+F 0 "R6" V 6000 3000 50  0000 L CNN
 F 1 "1Ω/1W" V 6000 3150 50  0000 L CNN
 F 2 "" V 6030 3200 50  0001 C CNN
@@
 $EndComp
 $Comp
-L Device:R R6
+L Device:R R7
 U 1 1 624C3E95
 P 6300 3200
-F 0 "R6" V 6200 3000 50  0000 L CNN
+F 0 "R7" V 6200 3000 50  0000 L CNN
 F 1 "1Ω/1W" V 6200 3150 50  0000 L CNN
 F 2 "" V 6230 3200 50  0001 C CNN
@@
 $EndComp
 $Comp
-L Device:R R7
+L Device:R R8
 U 1 1 624C41A7
 P 6500 3200
-F 0 "R7" V 6400 3000 50  0000 L CNN
+F 0 "R8" V 6400 3000 50  0000 L CNN
 F 1 "1Ω/1W" V 6400 3150 50  0000 L CNN
 F 2 "" V 6430 3200 50  0001 C CNN
@@
 	4550 1550 4325 1550
 $Comp
-L Device:R R3
+L Device:R R4
 U 1 1 62503BEE
 P 4775 2900
-F 0 "R3" V 4875 2775 50  0000 C CNN
+F 0 "R4" V 4875 2775 50  0000 C CNN
 F 1 "10kΩ" V 4875 2975 50  0000 C CNN
 F 2 "" V 4705 2900 50  0001 C CNN
@@
 	3875 2150 3875 2400
 $Comp
-L Device:R R2
+L Device:R R3
 U 1 1 6251750F
 P 3875 2550
-F 0 "R2" H 3945 2596 50  0000 L CNN
+F 0 "R3" H 3945 2596 50  0000 L CNN
 F 1 "2.2kΩ" H 3945 2505 50  0000 L CNN
 F 2 "" V 3805 2550 50  0001 C CNN
@@
 $EndComp
 $Comp
-L Device:C C3
-U 1 1 62678DAC
-P 3675 1650
-F 0 "C3" H 3790 1696 50  0000 L CNN
-F 1 "100nF" H 3790 1605 50  0000 L CNN
-F 2 "" H 3713 1500 50  0001 C CNN
-F 3 "~" H 3675 1650 50  0001 C CNN
-	1    3675 1650
-	1    0    0    -1
-$EndComp
-$Comp
 L power:GND #PWR07
 U 1 1 6267960D
@@
 $EndComp
 Wire Wire Line
-	3675 1850 3675 1800
-Wire Wire Line
 	3675 1500 3675 1450
 Wire Wire Line
@@
 Wire Wire Line
 	5550 2150 5900 2150
+$Comp
+L Device:R R2
+U 1 1 626540CC
+P 3675 1650
+F 0 "R2" H 3745 1696 50  0000 L CNN
+F 1 "330kΩ" H 3745 1605 50  0000 L CNN
+F 2 "" V 3605 1650 50  0001 C CNN
+F 3 "~" H 3675 1650 50  0001 C CNN
+	1    3675 1650
+	1    0    0    -1
+$EndComp
+Wire Wire Line
+	3675 1850 3675 1800
 $EndSCHEMATC

Commit message: Updated smart-pump
Parts:
- added R5: 1kΩ, symbol Device:R
- renumbered R5 to R6, R6 to R7, R7 to R8, R8 to R9
Connections:
- net at U2.12 (9*): now also R5.2; no longer Q1.4 (G)
- new net: Q1.4 (G), R5.1
Other:
- moved on the sheet: D2, Q1, R6, R7, R8, R9
Changed lines of the file:
@@
 Sheet 1 1
 Title "Smart Water Pump"
-Date "2022-04-24"
+Date "2022-04-25"
 Rev ""
 Comp "µF"
@@
 	1800 2225 1800 2200
 $Comp
-L Device:R R5
+L Device:R R6
 U 1 1 624BB180
-P 5900 3200
-F 0 "R5" V 5800 3000 50  0000 L CNN
-F 1 "1Ω/1W" V 5800 3150 50  0000 L CNN
-F 2 "" V 5830 3200 50  0001 C CNN
-F 3 "~" H 5900 3200 50  0001 C CNN
-	1    5900 3200
+P 6025 3200
+F 0 "R6" V 5925 3000 50  0000 L CNN
+F 1 "1Ω/1W" V 5925 3150 50  0000 L CNN
+F 2 "" V 5955 3200 50  0001 C CNN
+F 3 "~" H 6025 3200 50  0001 C CNN
+	1    6025 3200
 	1    0    0    -1
 $EndComp
@@
 	1800 2425 1800 2450
 $Comp
-L Device:R R6
+L Device:R R7
 U 1 1 624C399C
-P 6100 3200
-F 0 "R6" V 6000 3000 50  0000 L CNN
-F 1 "1Ω/1W" V 6000 3150 50  0000 L CNN
-F 2 "" V 6030 3200 50  0001 C CNN
-F 3 "~" H 6100 3200 50  0001 C CNN
-	1    6100 3200
-	1    0    0    -1
-$EndComp
-$Comp
-L Device:R R7
+P 6225 3200
+F 0 "R7" V 6125 3000 50  0000 L CNN
+F 1 "1Ω/1W" V 6125 3150 50  0000 L CNN
+F 2 "" V 6155 3200 50  0001 C CNN
+F 3 "~" H 6225 3200 50  0001 C CNN
+	1    6225 3200
+	1    0    0    -1
+$EndComp
+$Comp
+L Device:R R8
 U 1 1 624C3E95
-P 6300 3200
-F 0 "R7" V 6200 3000 50  0000 L CNN
-F 1 "1Ω/1W" V 6200 3150 50  0000 L CNN
-F 2 "" V 6230 3200 50  0001 C CNN
-F 3 "~" H 6300 3200 50  0001 C CNN
-	1    6300 3200
-	1    0    0    -1
-$EndComp
-$Comp
-L Device:R R8
+P 6425 3200
+F 0 "R8" V 6325 3000 50  0000 L CNN
+F 1 "1Ω/1W" V 6325 3150 50  0000 L CNN
+F 2 "" V 6355 3200 50  0001 C CNN
+F 3 "~" H 6425 3200 50  0001 C CNN
+	1    6425 3200
+	1    0    0    -1
+$EndComp
+$Comp
+L Device:R R9
 U 1 1 624C41A7
-P 6500 3200
-F 0 "R8" V 6400 3000 50  0000 L CNN
-F 1 "1Ω/1W" V 6400 3150 50  0000 L CNN
-F 2 "" V 6430 3200 50  0001 C CNN
-F 3 "~" H 6500 3200 50  0001 C CNN
-	1    6500 3200
-	1    0    0    -1
-$EndComp
-Wire Wire Line
-	5900 3050 5900 2900
-Wire Wire Line
-	5900 2900 6100 2900
-Wire Wire Line
-	6500 2900 6500 3050
-Wire Wire Line
-	6100 3050 6100 2900
-Connection ~ 6100 2900
-Wire Wire Line
-	6300 3050 6300 2900
-Connection ~ 6300 2900
-Wire Wire Line
-	6300 2900 6500 2900
-Wire Wire Line
-	5900 3350 5900 3475
-Wire Wire Line
-	5900 3475 6100 3475
-Wire Wire Line
-	6500 3475 6500 3350
-Wire Wire Line
-	6300 3350 6300 3475
-Connection ~ 6300 3475
-Wire Wire Line
-	6300 3475 6500 3475
-Wire Wire Line
-	6100 3350 6100 3475
-Connection ~ 6100 3475
-Wire Wire Line
-	6100 3475 6200 3475
+P 6625 3200
+F 0 "R9" V 6525 3000 50  0000 L CNN
+F 1 "1Ω/1W" V 6525 3150 50  0000 L CNN
+F 2 "" V 6555 3200 50  0001 C CNN
+F 3 "~" H 6625 3200 50  0001 C CNN
+	1    6625 3200
+	1    0    0    -1
+$EndComp
+Wire Wire Line
+	6025 3050 6025 2900
+Wire Wire Line
+	6025 2900 6225 2900
+Wire Wire Line
+	6625 2900 6625 3050
+Wire Wire Line
+	6225 3050 6225 2900
+Connection ~ 6225 2900
+Wire Wire Line
+	6425 3050 6425 2900
+Connection ~ 6425 2900
+Wire Wire Line
+	6425 2900 6625 2900
+Wire Wire Line
+	6025 3350 6025 3475
+Wire Wire Line
+	6025 3475 6225 3475
+Wire Wire Line
+	6625 3475 6625 3350
+Wire Wire Line
+	6425 3350 6425 3475
+Connection ~ 6425 3475
+Wire Wire Line
+	6425 3475 6625 3475
+Wire Wire Line
+	6225 3350 6225 3475
+Connection ~ 6225 3475
+Wire Wire Line
+	6225 3475 6325 3475
 $Comp
 L power:GND #PWR012
 U 1 1 624D1273
-P 6200 3575
-F 0 "#PWR012" H 6200 3325 50  0001 C CNN
-F 1 "GND" H 6205 3402 50  0000 C CNN
-F 2 "" H 6200 3575 50  0001 C CNN
-F 3 "" H 6200 3575 50  0001 C CNN
-	1    6200 3575
-	1    0    0    -1
-$EndComp
-Wire Wire Line
-	6200 3575 6200 3475
-Connection ~ 6200 3475
-Wire Wire Line
-	6200 3475 6300 3475
-Text GLabel 6575 1300 2    50   Output ~ 0
+P 6325 3575
+F 0 "#PWR012" H 6325 3325 50  0001 C CNN
+F 1 "GND" H 6330 3402 50  0000 C CNN
+F 2 "" H 6325 3575 50  0001 C CNN
+F 3 "" H 6325 3575 50  0001 C CNN
+	1    6325 3575
+	1    0    0    -1
+$EndComp
+Wire Wire Line
+	6325 3575 6325 3475
+Connection ~ 6325 3475
+Wire Wire Line
+	6325 3475 6425 3475
+Text GLabel 6700 1300 2    50   Output ~ 0
 M+
-Text GLabel 6575 1775 2    50   Output ~ 0
+Text GLabel 6700 1775 2    50   Output ~ 0
 M-
 Wire Wire Line
-	6200 1775 6575 1775
+	6325 1775 6700 1775
 $Comp
 L power:+12V #PWR011
 U 1 1 624EF9D8
-P 6200 1050
-F 0 "#PWR011" H 6200 900 50  0001 C CNN
-F 1 "+12V" H 6215 1223 50  0000 C CNN
-F 2 "" H 6200 1050 50  0001 C CNN
-F 3 "" H 6200 1050 50  0001 C CNN
-	1    6200 1050
+P 6325 1050
+F 0 "#PWR011" H 6325 900 50  0001 C CNN
+F 1 "+12V" H 6340 1223 50  0000 C CNN
+F 2 "" H 6325 1050 50  0001 C CNN
+F 3 "" H 6325 1050 50  0001 C CNN
+	1    6325 1050
 	1    0    0    -1
 $EndComp
@@
 L Diode:1N4007 D2
 U 1 1 624F2CB9
-P 6200 1525
-F 0 "D2" V 6154 1605 50  0000 L CNN
-F 1 "1N4007" V 6245 1605 50  0000 L CNN
-F 2 "Diode_THT:D_DO-41_SOD81_P10.16mm_Horizontal" H 6200 1350 50  0001 C CNN
-F 3 "http://www.vishay.com/docs/88503/1n4001.pdf" H 6200 1525 50  0001 C CNN
-	1    6200 1525
+P 6325 1525
+F 0 "D2" V 6279 1605 50  0000 L CNN
+F 1 "1N4007" V 6370 1605 50  0000 L CNN
+F 2 "Diode_THT:D_DO-41_SOD81_P10.16mm_Horizontal" H 6325 1350 50  0001 C CNN
+F 3 "http://www.vishay.com/docs/88503/1n4001.pdf" H 6325 1525 50  0001 C CNN
+	1    6325 1525
 	0    1    1    0
 $EndComp
 Wire Wire Line
-	6200 1775 6200 1675
-Wire Wire Line
-	6200 1375 6200 1300
-Wire Wire Line
-	6200 1300 6575 1300
-Connection ~ 6200 1300
+	6325 1775 6325 1675
+Wire Wire Line
+	6325 1375 6325 1300
+Wire Wire Line
+	6325 1300 6700 1300
+Connection ~ 6325 1300
 Wire Wire Line
 	4550 1550 4325 1550
@@
 	0    -1   -1   0
 $EndComp
-Text Notes 5750 2825 0    50   ~ 0
+Text Notes 5875 2825 0    50   ~ 0
 Shunt
 Wire Notes Line
-	5725 3550 6625 3550
+	5850 3550 6750 3550
 Wire Notes Line
-	6625 2725 5725 2725
+	6750 2725 5850 2725
 Wire Notes Line
-	6625 2725 6625 3550
+	6750 2725 6750 3550
 Wire Notes Line
-	5725 2725 5725 3550
+	5850 2725 5850 3550
 $Comp
 L power:+5V #PWR010
@@
 L Transistor_FET:IRF8721PBF-1 Q1
 U 1 1 626488E7
-P 6100 2150
-F 0 "Q1" H 6304 2196 50  0000 L CNN
-F 1 "IRF8721PBF" H 6304 2105 50  0000 L CNN
-F 2 "Package_SO:SOIC-8_3.9x4.9mm_P1.27mm" H 6300 2050 50  0001 L CNN
-F 3 "http://www.irf.com/product-info/datasheets/data/irf8721pbf-1.pdf" H 6100 2150 50  0001 L CNN
-	1    6100 2150
-	1    0    0    -1
-$EndComp
-Wire Wire Line
-	6100 2900 6200 2900
-Wire Wire Line
-	6200 1050 6200 1300
-Wire Wire Line
-	6200 1775 6200 1950
-Connection ~ 6200 1775
-Wire Wire Line
-	6200 2900 6200 2350
-Connection ~ 6200 2900
-Wire Wire Line
-	6200 2900 6300 2900
+P 6225 2150
+F 0 "Q1" H 6429 2196 50  0000 L CNN
+F 1 "IRF8721PBF" H 6429 2105 50  0000 L CNN
+F 2 "Package_SO:SOIC-8_3.9x4.9mm_P1.27mm" H 6425 2050 50  0001 L CNN
+F 3 "http://www.irf.com/product-info/datasheets/data/irf8721pbf-1.pdf" H 6225 2150 50  0001 L CNN
+	1    6225 2150
+	1    0    0    -1
+$EndComp
+Wire Wire Line
+	6225 2900 6325 2900
+Wire Wire Line
+	6325 1050 6325 1300
+Wire Wire Line
+	6325 1775 6325 1950
+Connection ~ 6325 1775
+Wire Wire Line
+	6325 2900 6325 2350
+Connection ~ 6325 2900
+Wire Wire Line
+	6325 2900 6425 2900
 $Comp
 L power:+5V #PWR06
@@
 Wire Wire Line
 	3675 1500 3675 1450
-Wire Wire Line
-	4925 2900 5900 2900
-Connection ~ 5900 2900
-Wire Wire Line
-	5550 2150 5900 2150
+Connection ~ 6025 2900
 $Comp
 L Device:R R2
@@
 Wire Wire Line
 	3675 1850 3675 1800
+$Comp
+L Device:R R5
+U 1 1 62666DD5
+P 5800 2150
+F 0 "R5" V 5900 2025 50  0000 C CNN
+F 1 "1kΩ" V 5900 2225 50  0000 C CNN
+F 2 "" V 5730 2150 50  0001 C CNN
+F 3 "~" H 5800 2150 50  0001 C CNN
+	1    5800 2150
+	0    1    1    0
+$EndComp
+Wire Wire Line
+	4925 2900 6025 2900
+Wire Wire Line
+	5550 2150 5650 2150
+Wire Wire Line
+	5950 2150 6025 2150
 $EndSCHEMATC

Commit message: Updated caravan
Connections:
- net +12V: now also J1.1 (Pin_1); no longer J1.3 (Pin_3)
- net GND: now also J1.2 (Pin_2); no longer J1.1 (Pin_1)
- net LEVEL: now also J1.3 (Pin_3); no longer J1.2 (Pin_2)
Changed lines of the file:
@@
 Sheet 1 1
 Title "Smart Water Pump"
-Date "2022-04-25"
+Date "2022-04-29"
 Rev ""
 Comp "µF"
@@
 	1500 1500 2075 1500
 $Comp
-L power:+12V #PWR02
-U 1 1 624B860C
-P 1800 2200
-F 0 "#PWR02" H 1800 2050 50  0001 C CNN
-F 1 "+12V" H 1815 2373 50  0000 C CNN
-F 2 "" H 1800 2200 50  0001 C CNN
-F 3 "" H 1800 2200 50  0001 C CNN
-	1    1800 2200
-	1    0    0    -1
-$EndComp
-Wire Wire Line
-	1700 2225 1800 2225
-Wire Wire Line
-	1800 2225 1800 2200
-$Comp
 L Device:R R6
 U 1 1 624BB180
@@
 Wire Wire Line
 	1700 2950 1900 2950
-Wire Wire Line
-	1700 2425 1800 2425
-Wire Wire Line
-	1800 2425 1800 2450
 $Comp
 L Device:R R7
@@
 	-1   0    0    1
 $EndComp
-Text GLabel 1900 2325 2    50   Output ~ 0
+Text GLabel 1900 2225 2    50   Output ~ 0
 LEVEL
-Wire Wire Line
-	1700 2325 1900 2325
 $Comp
 L power:GND #PWR03
 U 1 1 62675ECE
-P 1800 2450
-F 0 "#PWR03" H 1800 2200 50  0001 C CNN
-F 1 "GND" H 1805 2277 50  0000 C CNN
-F 2 "" H 1800 2450 50  0001 C CNN
-F 3 "" H 1800 2450 50  0001 C CNN
-	1    1800 2450
+P 2075 2475
+F 0 "#PWR03" H 2075 2225 50  0001 C CNN
+F 1 "GND" H 2080 2302 50  0000 C CNN
+F 2 "" H 2075 2475 50  0001 C CNN
+F 3 "" H 2075 2475 50  0001 C CNN
+	1    2075 2475
 	1    0    0    -1
 $EndComp
@@
 Wire Wire Line
 	5950 2150 6025 2150
+Wire Wire Line
+	1700 2225 1900 2225
+Wire Wire Line
+	1700 2425 1725 2425
+Wire Wire Line
+	1725 2425 1725 2650
+Wire Wire Line
+	1725 2650 1850 2650
+Wire Wire Line
+	1850 2650 1850 2625
+Wire Wire Line
+	1700 2325 2075 2325
+Wire Wire Line
+	2075 2325 2075 2475
+$Comp
+L power:+12V #PWR02
+U 1 1 624B860C
+P 1850 2625
+F 0 "#PWR02" H 1850 2475 50  0001 C CNN
+F 1 "+12V" H 1865 2798 50  0000 C CNN
+F 2 "" H 1850 2625 50  0001 C CNN
+F 3 "" H 1850 2625 50  0001 C CNN
+	1    1850 2625
+	1    0    0    -1
+$EndComp
 $EndSCHEMATC

Commit message: Updated smart-pump
Parts:
- added R5: 10kΩ, symbol Device:R
- renumbered R9 to R10, R5 to R6, R6 to R7, R7 to R8, R8 to R9
Connections:
- net GND: now also R5.2
- net at R6.2, U2.12 (9*): now also R5.1
Other:
- moved on the sheet: R6
Changed lines of the file:
@@
 Sheet 1 1
 Title "Smart Water Pump"
-Date "2022-04-29"
+Date "2022-04-30"
 Rev ""
 Comp "µF"
@@
 Connection ~ 1500 1150
 $Comp
-L power:GND #PWR04
+L power:GND #PWR03
 U 1 1 624AA5A3
 P 2075 1550
-F 0 "#PWR04" H 2075 1300 50  0001 C CNN
+F 0 "#PWR03" H 2075 1300 50  0001 C CNN
 F 1 "GND" H 2080 1377 50  0000 C CNN
 F 2 "" H 2075 1550 50  0001 C CNN
@@
 	1500 1500 2075 1500
 $Comp
-L Device:R R6
+L Device:R R7
 U 1 1 624BB180
 P 6025 3200
-F 0 "R6" V 5925 3000 50  0000 L CNN
+F 0 "R7" V 5925 3000 50  0000 L CNN
 F 1 "1Ω/1W" V 5925 3150 50  0000 L CNN
 F 2 "" V 5955 3200 50  0001 C CNN
@@
 	1700 2950 1900 2950
 $Comp
-L Device:R R7
+L Device:R R8
 U 1 1 624C399C
 P 6225 3200
-F 0 "R7" V 6125 3000 50  0000 L CNN
+F 0 "R8" V 6125 3000 50  0000 L CNN
 F 1 "1Ω/1W" V 6125 3150 50  0000 L CNN
 F 2 "" V 6155 3200 50  0001 C CNN
@@
 $EndComp
 $Comp
-L Device:R R8
+L Device:R R9
 U 1 1 624C3E95
 P 6425 3200
-F 0 "R8" V 6325 3000 50  0000 L CNN
+F 0 "R9" V 6325 3000 50  0000 L CNN
 F 1 "1Ω/1W" V 6325 3150 50  0000 L CNN
 F 2 "" V 6355 3200 50  0001 C CNN
@@
 $EndComp
 $Comp
-L Device:R R9
+L Device:R R10
 U 1 1 624C41A7
 P 6625 3200
-F 0 "R9" V 6525 3000 50  0000 L CNN
+F 0 "R10" V 6525 3000 50  0000 L CNN
 F 1 "1Ω/1W" V 6525 3150 50  0000 L CNN
 F 2 "" V 6555 3200 50  0001 C CNN
@@
 	6225 3475 6325 3475
 $Comp
-L power:GND #PWR012
+L power:GND #PWR013
 U 1 1 624D1273
 P 6325 3575
-F 0 "#PWR012" H 6325 3325 50  0001 C CNN
+F 0 "#PWR013" H 6325 3325 50  0001 C CNN
 F 1 "GND" H 6330 3402 50  0000 C CNN
 F 2 "" H 6325 3575 50  0001 C CNN
@@
 	6325 1775 6700 1775
 $Comp
-L power:+12V #PWR011
+L power:+12V #PWR012
 U 1 1 624EF9D8
 P 6325 1050
-F 0 "#PWR011" H 6325 900 50  0001 C CNN
+F 0 "#PWR012" H 6325 900 50  0001 C CNN
 F 1 "+12V" H 6340 1223 50  0000 C CNN
 F 2 "" H 6325 1050 50  0001 C CNN
@@
 LEVEL
 $Comp
-L power:GND #PWR03
+L power:GND #PWR04
 U 1 1 62675ECE
 P 2075 2475
-F 0 "#PWR03" H 2075 2225 50  0001 C CNN
+F 0 "#PWR04" H 2075 2225 50  0001 C CNN
 F 1 "GND" H 2080 2302 50  0000 C CNN
 F 2 "" H 2075 2475 50  0001 C CNN
@@
 	3675 1850 3675 1800
 $Comp
-L Device:R R5
+L Device:R R6
 U 1 1 62666DD5
-P 5800 2150
-F 0 "R5" V 5900 2025 50  0000 C CNN
-F 1 "1kΩ" V 5900 2225 50  0000 C CNN
-F 2 "" V 5730 2150 50  0001 C CNN
-F 3 "~" H 5800 2150 50  0001 C CNN
-	1    5800 2150
+P 5850 2150
+F 0 "R6" V 5950 2075 50  0000 C CNN
+F 1 "1kΩ" V 5950 2225 50  0000 C CNN
+F 2 "" V 5780 2150 50  0001 C CNN
+F 3 "~" H 5850 2150 50  0001 C CNN
+	1    5850 2150
 	0    1    1    0
 $EndComp
@@
 	4925 2900 6025 2900
 Wire Wire Line
-	5550 2150 5650 2150
-Wire Wire Line
-	5950 2150 6025 2150
+	5550 2150 5675 2150
+Wire Wire Line
+	6000 2150 6025 2150
 Wire Wire Line
 	1700 2225 1900 2225
@@
 	1    0    0    -1
 $EndComp
+$Comp
+L Device:R R5
+U 1 1 626D3BE6
+P 5675 2425
+F 0 "R5" H 5745 2471 50  0000 L CNN
+F 1 "10kΩ" H 5745 2380 50  0000 L CNN
+F 2 "" V 5605 2425 50  0001 C CNN
+F 3 "~" H 5675 2425 50  0001 C CNN
+	1    5675 2425
+	1    0    0    -1
+$EndComp
+Wire Wire Line
+	5675 2275 5675 2150
+Connection ~ 5675 2150
+Wire Wire Line
+	5675 2150 5700 2150
+$Comp
+L power:GND #PWR011
+U 1 1 626D6873
+P 5675 2600
+F 0 "#PWR011" H 5675 2350 50  0001 C CNN
+F 1 "GND" H 5680 2427 50  0000 C CNN
+F 2 "" H 5675 2600 50  0001 C CNN
+F 3 "" H 5675 2600 50  0001 C CNN
+	1    5675 2600
+	1    0    0    -1
+$EndComp
+Wire Wire Line
+	5675 2600 5675 2575
 $EndSCHEMATC
