File: smart-pump/smart-pump.sch (KiCad schematic (older format))
At the start: 21 parts, among them J1 Screw_Terminal_01x03, J2 Screw_Terminal_01x02, Q1 IRF8721PBF, SW1 SW_SPST, U1 AMS1117-5.0, U2 Arduino_Pro_Mini

Commit message: Updated smart pump
Parts:
- R1: value 1MΩ -> 4MΩ
- R2: value 330kΩ -> 1MΩ
Changed lines of the file:
@@
 Sheet 1 1
 Title "Smart Water Pump"
-Date "2022-04-30"
+Date "2022-05-02"
 Rev ""
 Comp "µF"
@@
 P 3675 1275
 F 0 "R1" H 3745 1321 50  0000 L CNN
-F 1 "1MΩ" H 3745 1230 50  0000 L CNN
+F 1 "4MΩ" H 3745 1230 50  0000 L CNN
 F 2 "" V 3605 1275 50  0001 C CNN
 F 3 "~" H 3675 1275 50  0001 C CNN
@@
 P 3675 1650
 F 0 "R2" H 3745 1696 50  0000 L CNN
-F 1 "330kΩ" H 3745 1605 50  0000 L CNN
+F 1 "1MΩ" H 3745 1605 50  0000 L CNN
 F 2 "" V 3605 1650 50  0001 C CNN
 F 3 "~" H 3675 1650 50  0001 C CNN

Commit message: Updated smart-pump
Parts:
- added R1: 10kΩ, symbol Device:R
- renumbered R9 to R10, R10 to R11, R1 to R2, R2 to R3, R3 to R4, R4 to R5, R5 to R6, R6 to R7, R7 to R8, R8 to R9
Connections:
- net LEVEL: now also R1.2; no longer R2.2, R3.1, U2.20 (A3)
- new net: R1.1, R2.2, R3.1, U2.20 (A3)
Other:
- moved on the sheet: R2, R3
Changed lines of the file:
@@
 Sheet 1 1
 Title "Smart Water Pump"
-Date "2022-05-02"
+Date "2022-05-03"
 Rev ""
 Comp "µF"
@@
 	1500 1500 2075 1500
 $Comp
-L Device:R R7
+L Device:R R8
 U 1 1 624BB180
 P 6025 3200
-F 0 "R7" V 5925 3000 50  0000 L CNN
+F 0 "R8" V 5925 3000 50  0000 L CNN
 F 1 "1Ω/1W" V 5925 3150 50  0000 L CNN
 F 2 "" V 5955 3200 50  0001 C CNN
@@
 	1700 2950 1900 2950
 $Comp
-L Device:R R8
+L Device:R R9
 U 1 1 624C399C
 P 6225 3200
-F 0 "R8" V 6125 3000 50  0000 L CNN
+F 0 "R9" V 6125 3000 50  0000 L CNN
 F 1 "1Ω/1W" V 6125 3150 50  0000 L CNN
 F 2 "" V 6155 3200 50  0001 C CNN
@@
 $EndComp
 $Comp
-L Device:R R9
+L Device:R R10
 U 1 1 624C3E95
 P 6425 3200
-F 0 "R9" V 6325 3000 50  0000 L CNN
+F 0 "R10" V 6325 3000 50  0000 L CNN
 F 1 "1Ω/1W" V 6325 3150 50  0000 L CNN
 F 2 "" V 6355 3200 50  0001 C CNN
@@
 $EndComp
 $Comp
-L Device:R R10
+L Device:R R11
 U 1 1 624C41A7
 P 6625 3200
-F 0 "R10" V 6525 3000 50  0000 L CNN
+F 0 "R11" V 6525 3000 50  0000 L CNN
 F 1 "1Ω/1W" V 6525 3150 50  0000 L CNN
 F 2 "" V 6555 3200 50  0001 C CNN
@@
 	4550 1550 4325 1550
 $Comp
-L Device:R R4
+L Device:R R5
 U 1 1 62503BEE
 P 4775 2900
-F 0 "R4" V 4875 2775 50  0000 C CNN
+F 0 "R5" V 4875 2775 50  0000 C CNN
 F 1 "10kΩ" V 4875 2975 50  0000 C CNN
 F 2 "" V 4705 2900 50  0001 C CNN
@@
 	3875 2150 3875 2400
 $Comp
-L Device:R R3
+L Device:R R4
 U 1 1 6251750F
 P 3875 2550
-F 0 "R3" H 3945 2596 50  0000 L CNN
+F 0 "R4" H 3945 2596 50  0000 L CNN
 F 1 "2.2kΩ" H 3945 2505 50  0000 L CNN
 F 2 "" V 3805 2550 50  0001 C CNN
@@
 $EndComp
 $Comp
-L Device:R R1
+L Device:R R2
 U 1 1 6255CFA6
-P 3675 1275
-F 0 "R1" H 3745 1321 50  0000 L CNN
-F 1 "4MΩ" H 3745 1230 50  0000 L CNN
-F 2 "" V 3605 1275 50  0001 C CNN
-F 3 "~" H 3675 1275 50  0001 C CNN
-	1    3675 1275
-	1    0    0    -1
-$EndComp
-Wire Wire Line
-	3675 1050 3675 1125
-Wire Wire Line
-	3675 1425 3675 1450
-Wire Wire Line
-	4550 1450 3675 1450
+P 3775 1275
+F 0 "R2" H 3845 1321 50  0000 L CNN
+F 1 "4MΩ" H 3845 1230 50  0000 L CNN
+F 2 "" V 3705 1275 50  0001 C CNN
+F 3 "~" H 3775 1275 50  0001 C CNN
+	1    3775 1275
+	1    0    0    -1
+$EndComp
+Wire Wire Line
+	3775 1050 3775 1125
+Wire Wire Line
+	3775 1425 3775 1450
 $Comp
 L Transistor_FET:IRF8721PBF-1 Q1
@@
 L power:+5V #PWR06
 U 1 1 62659641
-P 3675 1050
-F 0 "#PWR06" H 3675 900 50  0001 C CNN
-F 1 "+5V" H 3690 1223 50  0000 C CNN
-F 2 "" H 3675 1050 50  0001 C CNN
-F 3 "" H 3675 1050 50  0001 C CNN
-	1    3675 1050
-	1    0    0    -1
-$EndComp
-Text GLabel 3550 1450 0    50   Input ~ 0
+P 3775 1050
+F 0 "#PWR06" H 3775 900 50  0001 C CNN
+F 1 "+5V" H 3790 1223 50  0000 C CNN
+F 2 "" H 3775 1050 50  0001 C CNN
+F 3 "" H 3775 1050 50  0001 C CNN
+	1    3775 1050
+	1    0    0    -1
+$EndComp
+Text GLabel 3325 1450 0    50   Input ~ 0
 LEVEL
 Wire Wire Line
-	3550 1450 3675 1450
-Connection ~ 3675 1450
+	3675 1450 3775 1450
+Connection ~ 3775 1450
 $Comp
 L Connector:Screw_Terminal_01x03 J1
@@
 L power:GND #PWR07
 U 1 1 6267960D
-P 3675 1850
-F 0 "#PWR07" H 3675 1600 50  0001 C CNN
-F 1 "GND" H 3825 1775 50  0000 C CNN
-F 2 "" H 3675 1850 50  0001 C CNN
-F 3 "" H 3675 1850 50  0001 C CNN
-	1    3675 1850
-	1    0    0    -1
-$EndComp
-Wire Wire Line
-	3675 1500 3675 1450
+P 3775 1850
+F 0 "#PWR07" H 3775 1600 50  0001 C CNN
+F 1 "GND" H 3925 1775 50  0000 C CNN
+F 2 "" H 3775 1850 50  0001 C CNN
+F 3 "" H 3775 1850 50  0001 C CNN
+	1    3775 1850
+	1    0    0    -1
+$EndComp
+Wire Wire Line
+	3775 1500 3775 1450
 Connection ~ 6025 2900
 $Comp
-L Device:R R2
+L Device:R R3
 U 1 1 626540CC
-P 3675 1650
-F 0 "R2" H 3745 1696 50  0000 L CNN
-F 1 "1MΩ" H 3745 1605 50  0000 L CNN
-F 2 "" V 3605 1650 50  0001 C CNN
-F 3 "~" H 3675 1650 50  0001 C CNN
-	1    3675 1650
-	1    0    0    -1
-$EndComp
-Wire Wire Line
-	3675 1850 3675 1800
-$Comp
-L Device:R R6
+P 3775 1650
+F 0 "R3" H 3845 1696 50  0000 L CNN
+F 1 "1MΩ" H 3845 1605 50  0000 L CNN
+F 2 "" V 3705 1650 50  0001 C CNN
+F 3 "~" H 3775 1650 50  0001 C CNN
+	1    3775 1650
+	1    0    0    -1
+$EndComp
+Wire Wire Line
+	3775 1850 3775 1800
+$Comp
+L Device:R R7
 U 1 1 62666DD5
 P 5850 2150
-F 0 "R6" V 5950 2075 50  0000 C CNN
+F 0 "R7" V 5950 2075 50  0000 C CNN
 F 1 "1kΩ" V 5950 2225 50  0000 C CNN
 F 2 "" V 5780 2150 50  0001 C CNN
@@
 $EndComp
 $Comp
-L Device:R R5
+L Device:R R6
 U 1 1 626D3BE6
 P 5675 2425
-F 0 "R5" H 5745 2471 50  0000 L CNN
+F 0 "R6" H 5745 2471 50  0000 L CNN
 F 1 "10kΩ" H 5745 2380 50  0000 L CNN
 F 2 "" V 5605 2425 50  0001 C CNN
@@
 Wire Wire Line
 	5675 2600 5675 2575
+$Comp
+L Device:R R1
+U 1 1 62711193
+P 3525 1450
+F 0 "R1" V 3625 1350 50  0000 C CNN
+F 1 "10kΩ" V 3625 1525 50  0000 C CNN
+F 2 "" V 3455 1450 50  0001 C CNN
+F 3 "~" H 3525 1450 50  0001 C CNN
+	1    3525 1450
+	0    1    1    0
+$EndComp
+Wire Wire Line
+	4550 1450 3775 1450
+Wire Wire Line
+	3325 1450 3375 1450
 $EndSCHEMATC

Commit message: Updated smart-pump
Parts:
- removed R1: 10kΩ, symbol Device:R
- added C3: 470nF, symbol Device:C
- R1: renamed from R2; value 4MΩ -> 1MΩ
- R2: renamed from R3; value 1MΩ -> 270kΩ
- renumbered C3 to C4, R11 to R10, R4 to R3, R5 to R4, R6 to R5, R7 to R6, R8 to R7, R9 to R8, R10 to R9
Connections:
- net +5V: no longer R1.1
- net LEVEL: now also C3.1
- net at U2.11 (8): now also R1.1
- net at R1.2, R2.1, U2.20 (A3): now also C3.2
Other:
- moved on the sheet: R1
Changed lines of the file:
@@
 $EndComp
 $Comp
-L Device:C C3
+L Device:C C4
 U 1 1 624A13A7
 P 4325 3200
-F 0 "C3" H 4440 3246 50  0000 L CNN
+F 0 "C4" H 4440 3246 50  0000 L CNN
 F 1 "100nF" H 4440 3155 50  0000 L CNN
 F 2 "" H 4363 3050 50  0001 C CNN
@@
 	1500 1500 2075 1500
 $Comp
-L Device:R R8
+L Device:R R7
 U 1 1 624BB180
 P 6025 3200
-F 0 "R8" V 5925 3000 50  0000 L CNN
+F 0 "R7" V 5925 3000 50  0000 L CNN
 F 1 "1Ω/1W" V 5925 3150 50  0000 L CNN
 F 2 "" V 5955 3200 50  0001 C CNN
@@
 	1700 2950 1900 2950
 $Comp
-L Device:R R9
+L Device:R R8
 U 1 1 624C399C
 P 6225 3200
-F 0 "R9" V 6125 3000 50  0000 L CNN
+F 0 "R8" V 6125 3000 50  0000 L CNN
 F 1 "1Ω/1W" V 6125 3150 50  0000 L CNN
 F 2 "" V 6155 3200 50  0001 C CNN
@@
 $EndComp
 $Comp
-L Device:R R10
+L Device:R R9
 U 1 1 624C3E95
 P 6425 3200
-F 0 "R10" V 6325 3000 50  0000 L CNN
+F 0 "R9" V 6325 3000 50  0000 L CNN
 F 1 "1Ω/1W" V 6325 3150 50  0000 L CNN
 F 2 "" V 6355 3200 50  0001 C CNN
@@
 $EndComp
 $Comp
-L Device:R R11
+L Device:R R10
 U 1 1 624C41A7
 P 6625 3200
-F 0 "R11" V 6525 3000 50  0000 L CNN
+F 0 "R10" V 6525 3000 50  0000 L CNN
 F 1 "1Ω/1W" V 6525 3150 50  0000 L CNN
 F 2 "" V 6555 3200 50  0001 C CNN
@@
 	6225 3475 6325 3475
 $Comp
-L power:GND #PWR013
+L power:GND #PWR012
 U 1 1 624D1273
 P 6325 3575
-F 0 "#PWR013" H 6325 3325 50  0001 C CNN
+F 0 "#PWR012" H 6325 3325 50  0001 C CNN
 F 1 "GND" H 6330 3402 50  0000 C CNN
 F 2 "" H 6325 3575 50  0001 C CNN
@@
 	6325 1775 6700 1775
 $Comp
-L power:+12V #PWR012
+L power:+12V #PWR011
 U 1 1 624EF9D8
 P 6325 1050
-F 0 "#PWR012" H 6325 900 50  0001 C CNN
+F 0 "#PWR011" H 6325 900 50  0001 C CNN
 F 1 "+12V" H 6340 1223 50  0000 C CNN
 F 2 "" H 6325 1050 50  0001 C CNN
@@
 	4550 1550 4325 1550
 $Comp
-L Device:R R5
+L Device:R R4
 U 1 1 62503BEE
 P 4775 2900
-F 0 "R5" V 4875 2775 50  0000 C CNN
+F 0 "R4" V 4875 2775 50  0000 C CNN
 F 1 "10kΩ" V 4875 2975 50  0000 C CNN
 F 2 "" V 4705 2900 50  0001 C CNN
@@
 	4325 2900 4325 3050
 $Comp
-L power:GND #PWR09
+L power:GND #PWR08
 U 1 1 62508748
 P 4325 3575
-F 0 "#PWR09" H 4325 3325 50  0001 C CNN
+F 0 "#PWR08" H 4325 3325 50  0001 C CNN
 F 1 "GND" H 4330 3402 50  0000 C CNN
 F 2 "" H 4325 3575 50  0001 C CNN
@@
 	3875 2150 3875 2400
 $Comp
-L Device:R R4
+L Device:R R3
 U 1 1 6251750F
 P 3875 2550
-F 0 "R4" H 3945 2596 50  0000 L CNN
+F 0 "R3" H 3945 2596 50  0000 L CNN
 F 1 "2.2kΩ" H 3945 2505 50  0000 L CNN
 F 2 "" V 3805 2550 50  0001 C CNN
@@
 	5850 2725 5850 3550
 $Comp
-L power:+5V #PWR010
+L power:+5V #PWR09
 U 1 1 6253FA6A
 P 4400 1050
-F 0 "#PWR010" H 4400 900 50  0001 C CNN
+F 0 "#PWR09" H 4400 900 50  0001 C CNN
 F 1 "+5V" H 4415 1223 50  0000 C CNN
 F 2 "" H 4400 1050 50  0001 C CNN
@@
 	4400 1350 4550 1350
 $Comp
-L power:GND #PWR08
+L power:GND #PWR07
 U 1 1 625417BF
 P 4175 1225
-F 0 "#PWR08" H 4175 975 50  0001 C CNN
+F 0 "#PWR07" H 4175 975 50  0001 C CNN
 F 1 "GND" H 4180 1052 50  0000 C CNN
 F 2 "" H 4175 1225 50  0001 C CNN
@@
 $EndComp
 $Comp
-L Device:R R2
+L Device:R R1
 U 1 1 6255CFA6
-P 3775 1275
-F 0 "R2" H 3845 1321 50  0000 L CNN
-F 1 "4MΩ" H 3845 1230 50  0000 L CNN
-F 2 "" V 3705 1275 50  0001 C CNN
-F 3 "~" H 3775 1275 50  0001 C CNN
-	1    3775 1275
-	1    0    0    -1
-$EndComp
-Wire Wire Line
-	3775 1050 3775 1125
-Wire Wire Line
-	3775 1425 3775 1450
+P 3775 1250
+F 0 "R1" H 3845 1296 50  0000 L CNN
+F 1 "1MΩ" H 3845 1205 50  0000 L CNN
+F 2 "" V 3705 1250 50  0001 C CNN
+F 3 "~" H 3775 1250 50  0001 C CNN
+	1    3775 1250
+	1    0    0    -1
+$EndComp
+Wire Wire Line
+	3775 1400 3775 1450
 $Comp
 L Transistor_FET:IRF8721PBF-1 Q1
@@
 Wire Wire Line
 	6325 2900 6425 2900
-$Comp
-L power:+5V #PWR06
-U 1 1 62659641
-P 3775 1050
-F 0 "#PWR06" H 3775 900 50  0001 C CNN
-F 1 "+5V" H 3790 1223 50  0000 C CNN
-F 2 "" H 3775 1050 50  0001 C CNN
-F 3 "" H 3775 1050 50  0001 C CNN
-	1    3775 1050
-	1    0    0    -1
-$EndComp
 Text GLabel 3325 1450 0    50   Input ~ 0
 LEVEL
@@
 $EndComp
 $Comp
-L power:GND #PWR07
+L power:GND #PWR06
 U 1 1 6267960D
 P 3775 1850
-F 0 "#PWR07" H 3775 1600 50  0001 C CNN
+F 0 "#PWR06" H 3775 1600 50  0001 C CNN
 F 1 "GND" H 3925 1775 50  0000 C CNN
 F 2 "" H 3775 1850 50  0001 C CNN
@@
 Connection ~ 6025 2900
 $Comp
-L Device:R R3
+L Device:R R2
 U 1 1 626540CC
 P 3775 1650
-F 0 "R3" H 3845 1696 50  0000 L CNN
-F 1 "1MΩ" H 3845 1605 50  0000 L CNN
+F 0 "R2" H 3845 1696 50  0000 L CNN
+F 1 "270kΩ" H 3845 1605 50  0000 L CNN
 F 2 "" V 3705 1650 50  0001 C CNN
 F 3 "~" H 3775 1650 50  0001 C CNN
@@
 	3775 1850 3775 1800
 $Comp
-L Device:R R7
+L Device:R R6
 U 1 1 62666DD5
 P 5850 2150
-F 0 "R7" V 5950 2075 50  0000 C CNN
+F 0 "R6" V 5950 2075 50  0000 C CNN
 F 1 "1kΩ" V 5950 2225 50  0000 C CNN
 F 2 "" V 5780 2150 50  0001 C CNN
@@
 $EndComp
 $Comp
-L Device:R R6
+L Device:R R5
 U 1 1 626D3BE6
 P 5675 2425
-F 0 "R6" H 5745 2471 50  0000 L CNN
+F 0 "R5" H 5745 2471 50  0000 L CNN
 F 1 "10kΩ" H 5745 2380 50  0000 L CNN
 F 2 "" V 5605 2425 50  0001 C CNN
@@
 	5675 2150 5700 2150
 $Comp
-L power:GND #PWR011
+L power:GND #PWR010
 U 1 1 626D6873
 P 5675 2600
-F 0 "#PWR011" H 5675 2350 50  0001 C CNN
+F 0 "#PWR010" H 5675 2350 50  0001 C CNN
 F 1 "GND" H 5680 2427 50  0000 C CNN
 F 2 "" H 5675 2600 50  0001 C CNN
@@
 Wire Wire Line
 	5675 2600 5675 2575
-$Comp
-L Device:R R1
-U 1 1 62711193
+Wire Wire Line
+	4550 1450 3775 1450
+Wire Wire Line
+	3325 1450 3375 1450
+$Comp
+L Device:C C3
+U 1 1 6271AE39
 P 3525 1450
-F 0 "R1" V 3625 1350 50  0000 C CNN
-F 1 "10kΩ" V 3625 1525 50  0000 C CNN
-F 2 "" V 3455 1450 50  0001 C CNN
+F 0 "C3" V 3375 1525 50  0000 L CNN
+F 1 "470nF" V 3375 1275 50  0000 L CNN
+F 2 "" H 3563 1300 50  0001 C CNN
 F 3 "~" H 3525 1450 50  0001 C CNN
 	1    3525 1450
-	0    1    1    0
-$EndComp
-Wire Wire Line
-	4550 1450 3775 1450
-Wire Wire Line
-	3325 1450 3375 1450
+	0    -1   -1   0
+$EndComp
+Wire Wire Line
+	3775 700  5675 700
+Wire Wire Line
+	5675 700  5675 2050
+Wire Wire Line
+	5675 2050 5550 2050
+Wire Wire Line
+	3775 700  3775 1100
 $EndSCHEMATC
