File: tcs-intercom/tcs-intercom.kicad_sch (KiCad schematic)
At the start: 13 parts

Commit message: Updated tcs-intercom
Parts:
- removed J?: Screw_Terminal_01x02, symbol Connector:Screw_Terminal_01x02
- added J1: Screw_Terminal_01x04, symbol Connector:Screw_Terminal_01x04
- gave numbers to parts that had none: 12
Connections:
- net GND: now also J1.2 (Pin_2)
- net a: now also J1.1 (Pin_1)
- new net E: J1.3 (Pin_3)
- new net P: J1.4 (Pin_4)
Other:
- moved on the sheet: Q1, R1, R4

Commit message: Updated tcs-intercom
Parts:
- removed C2: 10µF, symbol Device:C_Polarized
- R1: value 0.5R 1W -> 27R
- R3: value 160K -> 150K
- R4: value 10K -> 1K

Commit message: Updated tcs-intercom
Connections:
- net P: now also D1.2 (A)
- net a: no longer D1.2 (A)
Other:
- note added: "Bus"
- note removed: "TCS Bus"
Changed lines of the file:
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@@
   (title_block
     (title "TCS Intercom Controller")
-    (date "2023-05-18")
+    (date "2023-05-19")
     (company "µF")
     (comment 1 "www.github.com/microfarad-de/tcs-intercom")
@@
   )
   (wire (pts (xy 78.74 87.63) (xy 81.28 87.63))
+    (stroke (width 0) (type default) (color 0 0 0 0))
+  )
+  (wire (pts (xy 63.5 63.5) (xy 63.5 33.02))
     (stroke (width 0) (type default) (color 0 0 0 0))
   )
@@
     (stroke (width 0) (type default) (color 0 0 0 0))
   )
-  (wire (pts (xy 55.88 63.5) (xy 59.055 63.5))
+  (wire (pts (xy 55.88 63.5) (xy 63.5 63.5))
     (stroke (width 0) (type default) (color 0 0 0 0))
   )
   (wire (pts (xy 120.015 62.23) (xy 120.015 72.39))
+    (stroke (width 0) (type default) (color 0 0 0 0))
+  )
+  (wire (pts (xy 63.5 33.02) (xy 81.28 33.02))
     (stroke (width 0) (type default) (color 0 0 0 0))
   )
@@
   )
   (wire (pts (xy 113.03 29.845) (xy 113.03 33.02))
-    (stroke (width 0) (type default) (color 0 0 0 0))
-  )
-  (wire (pts (xy 78.74 33.02) (xy 78.74 55.88))
     (stroke (width 0) (type default) (color 0 0 0 0))
   )
@@
     (stroke (width 0) (type default) (color 0 0 0 0))
   )
-  (wire (pts (xy 78.74 33.02) (xy 81.28 33.02))
-    (stroke (width 0) (type default) (color 0 0 0 0))
-  )
   (wire (pts (xy 106.68 87.63) (xy 108.585 87.63))
     (stroke (width 0) (type default) (color 0 0 0 0))
@@
     (stroke (width 0) (type default) (color 0 0 0 0))
   )
-  (text "TCS Bus" (at 40.005 57.785 0)
+  (text "Bus" (at 44.45 60.325 0)
     (effects (font (size 1.27 1.27)) (justify left bottom))
   )

Commit message: Updated tcs-intercom
Parts:
- added C2: 1000µF 10V, symbol Device:C_Polarized
- added C3: 470nF, symbol Device:C
- added J2: HC-05 Bluetooth, symbol Connector:Conn_01x06_Female
- added R7: 1K, symbol Device:R
- added R8: 2K2, symbol Device:R
- added R9: 22R, symbol Device:R
Connections:
- new net: C2.2, C3.2, J2.4 (Pin_4), R8.1, U2. (VCC)
- new net: J2.2 (Pin_2), R7.1, R8.2
- new net: C2.1, C3.1, J2.5 (Pin_5), R9.2
- new net: J2.3 (Pin_3), U2. (VCC)
- new net: R9.1, U2. (VCC)
- new net: R7.2, U2. (VCC)
Other:
- note added: "EN"
- note added: "GND"
- note added: "RXD"
- note added: "STATE"
- note added: "TXD"
- note added: "VCC"
- moved on the sheet: C1, D1, J1, Q1, R1, R2, R3, R4, R5, R6, U1
