File: delay-timer/delay-timer.kicad_sch (KiCad schematic)
At the start: 9 parts, among them J1 Input, J2 Output, U1 NE555D

Commit message: Updated delay-timer
Parts:
- R2: value 3.4MΩ -> 1MΩ
Other:
- note added: "Time delay in seconds t = R * C * ln(3) The current circuit has a delay of approx. 2 minutes for R2 = 1 MΩ and C3 = 100 µF"
- note removed: "3.4MΩ / 100µF provide a power on delay of approx. 7 minutes."
Changed lines of the file:
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@@
   (title_block
     (title "555 Delay Timer")
-    (date "2024-09-29")
+    (date "2024-10-12")
     (company "Copyright (C) 2024, Karim Hraibi")
     (comment 2 "by a time duration defined by the values of R2 and C3.")
@@
     (effects (font (size 1.27 1.27)) (justify left bottom))
   )
-  (text "3.4MΩ / 100µF provide \na power on delay of \napprox. 7 minutes."
-    (at 130.175 74.93 0)
+  (text "Time delay in seconds\nt = R * C * ln(3)\nThe current circuit has a \ndelay of approx. 2 minutes\nfor R2 = 1 MΩ and C3 = 100 µF "
+    (at 135.89 76.835 0)
     (effects (font (size 1.27 1.27)) (justify left bottom))
   )
@@
       (effects (font (size 1.27 1.27)) (justify left))
     )
-    (property "Value" "3.4MΩ" (id 1) (at 121.793 49.9622 0)
+    (property "Value" "1MΩ" (id 1) (at 121.793 49.9622 0)
       (effects (font (size 1.27 1.27)) (justify left))
     )
@@
     )
     (path "/b74d8b92-e4d4-45a9-93ff-ee3d3a9df3f3"
-      (reference "R2") (unit 1) (value "3.4MΩ") (footprint "")
+      (reference "R2") (unit 1) (value "1MΩ") (footprint "")
     )
     (path "/8910fa7f-b124-484f-8582-c326523d5863"
