File: 555-delay-advanced-2/555-delay-advanced-2.kicad_sch (KiCad schematic)
At the start: 15 parts, among them J1 Input, J2 Output, Q1 BC337, Q2 BC327, U1 NE555D

Commit message: Updated 555-delay-advanced-2
Parts:
- removed D1: 1N5819, Diode_THT:D_DO-41_SOD81_P10.16mm_Horizontal, symbol Diode:1N5819
- added D1: 1N4151, Diode_THT:D_DO-35_SOD27_P7.62mm_Horizontal, symbol Diode:1N4151
- added D2: 5.1V, symbol Device:D_Zener
- renumbered D2 to D3
Connections:
- net +12V: now also U1.6 (THR); no longer U1.4 (R)
- net GND: now also D1.1 (K)
- net at C1.1, R2.2, R3.2: now also U1.3 (Q); no longer U1.2 (TR)
- net at C2.1: now also U1.7 (DIS); no longer U1.5 (CV)
- net at R1.1: now also D1.2 (A), D2.1 (K); no longer Q1.2 (B)
- net at R4.2: now also U1.2 (TR); no longer U1.3 (Q)
- net at C3.1, R5.2: now also U1.4 (R), U1.5 (CV); no longer U1.6 (THR), U1.7 (DIS)
- new net: D2.2 (A), Q1.2 (B)
Other:
- moved on the sheet: J1, R1

Commit message: Updated 555-delay-advanced-2
Connections:
- net +12V: now also U1.4 (R); no longer U1.6 (THR)
- net at C1.1, R2.2, R3.2: now also U1.2 (TR); no longer U1.3 (Q)
- net at C2.1: now also U1.5 (CV); no longer U1.7 (DIS)
- net at R4.2: now also U1.3 (Q); no longer U1.2 (TR)
- net at C3.1, R5.2: now also U1.6 (THR), U1.7 (DIS); no longer U1.4 (R), U1.5 (CV)
Changed lines of the file:
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@@
     (pin "2")
   )
-  (symbol (lib_id "Timer:NE555D") (at 98.425 60.325 0) (mirror y) (unit 1)
+  (symbol (lib_id "Timer:NE555D") (at 98.425 60.325 0) (unit 1)
     (in_bom yes) (on_board yes) (fields_autoplaced)
-    (property "Reference" "U1" (id 0) (at 98.9456 49.0052 0)
-      (effects (font (size 1.27 1.27)) (justify right))
+    (property "Reference" "U1" (id 0) (at 100.4444 49.0052 0)
+      (effects (font (size 1.27 1.27)) (justify left))
     )
-    (property "Value" "NE555D" (id 1) (at 98.9456 51.5421 0)
-      (effects (font (size 1.27 1.27)) (justify right))
+    (property "Value" "NE555D" (id 1) (at 100.4444 51.5421 0)
+      (effects (font (size 1.27 1.27)) (justify left))
     )
-    (property "Footprint" "Package_SO:SOIC-8_3.9x4.9mm_P1.27mm" (id 2) (at 76.835 70.485 0)
+    (property "Footprint" "Package_SO:SOIC-8_3.9x4.9mm_P1.27mm" (id 2) (at 120.015 70.485 0)
       (effects (font (size 1.27 1.27)) hide)
     )
-    (property "Datasheet" "http://www.ti.com/lit/ds/symlink/ne555.pdf" (id 3) (at 76.835 70.485 0)
+    (property "Datasheet" "http://www.ti.com/lit/ds/symlink/ne555.pdf" (id 3) (at 120.015 70.485 0)
       (effects (font (size 1.27 1.27)) hide)
     )

Commit message: Updated 555-delay-advanced-2
Parts:
- removed D3: 1N4007, Diode_THT:D_DO-41_SOD81_P10.16mm_Horizontal, symbol Diode:1N4007
- added C1: 220µF, symbol Device:C_Polarized
- added D3: 1N4151, Diode_THT:D_DO-35_SOD27_P7.62mm_Horizontal, symbol Diode:1N4151
- C2: renamed from C1; value 100nF -> 470nF
- R1: value 47KΩ -> 10KΩ
- R3: value 100KΩ -> 47KΩ
- renumbered C2 to C3, C3 to C4
Connections:
- net +12V: now also C1.1, D3.1 (K)
- net GND: now also C1.2, D3.2 (A)
Other:
- note added: "This circuit ensures that the output is turned off for a minium time duration determined by R5/C4 (4MΩ/100µF = 8m 30s)"
- note removed: "This circuit ensures that the output is turned off for a minium time duration determined by R5/C3 (4MΩ/100µF = 8m 30s)"
- moved on the sheet: C2, C3, C4, D1, D2, J1, J2, Q1, Q2, R1, R2, R3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
