File: 555-delay-opto/555-delay-opto.kicad_sch (KiCad schematic)
At the start: 13 parts, among them U1 NE555D, U2 SFH6156-2

Commit message: Added fridge-controller
Parts:
- R5: value 470Ω -> 1KΩ
Changed lines of the file:
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@@
       (effects (font (size 1.27 1.27)) (justify left))
     )
-    (property "Value" "470Ω" (id 1) (at 145.923 49.9622 0)
+    (property "Value" "1KΩ" (id 1) (at 145.923 49.9622 0)
       (effects (font (size 1.27 1.27)) (justify left))
     )
@@
     )
     (path "/52a0c124-2aad-49b4-9ae6-f7669ee07272"
-      (reference "R5") (unit 1) (value "470Ω") (footprint "")
+      (reference "R5") (unit 1) (value "1KΩ") (footprint "")
     )
     (path "/8910fa7f-b124-484f-8582-c326523d5863"
